File: Hardware/AD9833FunctionGenerator.sch (KiCad schematic (older format))
At the start: 21 parts

Commit message: updated sw
- added five simultaneous ADC interrupts
- added mode, freq and sweep info to display
- added 7805 regulator for +/-12V and +5V rails.
Parts:
- removed C_REGIN1: 100uF, symbol CP
- removed C_REGOUT1, C_RIP1: CP, symbol CP
- removed D_REG1: 1N5819, symbol D_Schottky
- removed L_REG1: 100uH, symbol L_Core_Iron
- removed R_REG1, R_REG2, R_SC1: R, symbol R
- removed U_5VREG1: L7805, symbol L7805
- removed U_DIV1: MCP41010, symbol MCP41010
- removed U_INVREG1: MC34063, symbol MC34063
- added J_AMP1, J_FREQ2, J_OFFSET1, J_VEL1: Conn_01x03, symbol AD9833FunctionGenerator-rescue:Conn_01x03
- added R_FUNC1, R_MODE1, R_VEL1: 1K, symbol Device:R
- added SW_FUNC1, SW_MODE1: SW_SPST, symbol Switch:SW_SPST
- added U?: LM7805_TO220, Package_TO_SOT_THT:TO-220-3_Vertical, symbol Regulator_Linear:LM7805_TO220
- added U?: MCP42050, symbol Potentiometer_Digital:MCP42050
- C? (x2): symbol CP -> Device:CP
- J_AD9833: symbol Conn_01x07 -> AD9833FunctionGenerator-rescue:Conn_01x07
- J_FREQ1: symbol Conn_01x03 -> AD9833FunctionGenerator-rescue:Conn_01x03
- J_OLED1: symbol Conn_01x04 -> AD9833FunctionGenerator-rescue:Conn_01x04
- J_PWR1: symbol Conn_01x02 -> AD9833FunctionGenerator-rescue:Conn_01x02
- J_TX1, J_VIN: symbol Conn_01x15 -> AD9833FunctionGenerator-rescue:Conn_01x15
- R_DIV1: symbol R -> Device:R
- U_GAIN1: symbol TL072 -> AD9833FunctionGenerator-rescue:TL072
Connections:
- net labels added: AMP1, FREQ1, FREQ2, FUNC1, MODE1, OFFSET1, VEL1
- wire segments 79 -> 101
- no-connect marks 1 -> 2
Other:
- note added: "Direct Digital Synthesis Molex socket"
- note added: "OLED Display Molex socket"
- note added: "Output section"
- note added: "Potentiometer Molex Sockets"
- note added: "Power supply"
- note added: "SPST Molex Sockets"
- note added: "VIN\nGND\nRST\n5V\nA7\nA6\nA5\nA4\nA3\nA2\nA1\nA0\nAREF\n3V3\n13"
- note removed: "VIN\nGND\nRST\n5V\n21\n20\n19\n18\n17\n16\n15\n14\nAREF\n3V3\n13"

Commit message: updated
Connections:
- net labels added: DDS_CS, POT_CS
- net labels removed: CS
- wire segments 101 -> 109
Other:
- note added: "Arduino Nano sockets"
- note added: "TX\nRX\nRST\nGND\nD2\nD3\nD4\nD5\nD6\nD7\nD8\nD9\nD10\nD11\nD12"
- note added: "VIN\nGND\nRST\n5V\nA7\nA6\nA5\nA4\nA3\nA2\nA1\nA0\nAREF\n3V3\nD13"
- note removed: "TX\nRX\nRST\nGND\n2\n3\n4\n5\n6\n7\n8\n9\n10\n11\n12"
- note removed: "VIN\nGND\nRST\n5V\nA7\nA6\nA5\nA4\nA3\nA2\nA1\nA0\nAREF\n3V3\n13"

Commit message: fixed digpot/dds sidebyside spi config
Parts:
- removed J_PWR1: Conn_01x02, symbol AD9833FunctionGenerator-rescue:Conn_01x02
- removed R_DIV1: 82K, symbol Device:R
- removed U_GAIN1: TL072, symbol AD9833FunctionGenerator-rescue:TL072
- added J_PWR1: Conn_01x03, symbol Connector_Generic:Conn_01x03
- added R_ATTEN11, R_MIX1, R_MIX2, R_OFFSET1: 1K, symbol Device:R
- added U_OUTPUT1: TL074, symbol Amplifier_Operational:TL074
- gave numbers to parts that had none: 1
Connections:
- net labels added: FUNCSIGOUT, OUTPUT, SIGPOTOUT
- net labels removed: SIGOUT
- wire segments 109 -> 117
- no-connect marks 2 -> 5
Other:
- moved on the sheet: U_DIGPOT1

Commit message: added attenuation and amplitude opamp circuit
Parts:
- removed J_OFFSET1: Conn_01x03, symbol AD9833FunctionGenerator-rescue:Conn_01x03
- removed R_ATTEN11, R_MIX1, R_MIX2, R_OFFSET1: 1K, symbol Device:R
- removed unit 1 of U_OUTPUT1
- removed unit 2 of U_OUTPUT1
- added R_AMP1: 470R, symbol Device:R
- added R_ATEN1: 10K, symbol Device:R
Connections:
- net labels added: SIGFUNC
- net labels removed: AMP1, FUNCSIGOUT, OFFSET1, OUTPUT, SIGPOTOUT
- wire segments 117 -> 107
- no-connect marks 5 -> 2
Other:
- note added: "10K POT\n"
- note removed: "Output section"
- moved on the sheet: U_DIGPOT1, U_OUTPUT1C, U_OUTPUT1D, U_OUTPUT1E

Commit message: added analog output section for fixed gain compensation, variable offset and variable adjustments
Parts:
- removed J_AMP1: Conn_01x03, symbol AD9833FunctionGenerator-rescue:Conn_01x03
- removed R_ATEN1: 10K, symbol Device:R
- removed U_DIGPOT1: MCP42050, symbol Potentiometer_Digital:MCP42050
- removed U_OUTPUT1: TL074, symbol Amplifier_Operational:TL074
- added J_AMP1, J_OFFSET1: Conn_01x03, symbol Connector_Generic:Conn_01x03
- added RB1: 8K2, symbol Device:R
- added RB2, R_MIX1, R_MIX2: 1K, symbol Device:R
- added R_AF1: 15K, symbol Device:R
- added R_AG1: 1K2, symbol Device:R
- added R_AMP2: 470R, symbol Device:R
- added U? (x2): TL072, symbol AD9833FunctionGenerator-rescue:TL072
- added U_OUTPUT1: OPA1641, symbol Amplifier_Operational:OPA1641
- R_AMP1: value 470R -> 1K8
Connections:
- net labels added: +12V, OUTPUT
- net labels removed: 12V
- wire segments 107 -> 116
- no-connect marks 2 -> 1
Other:
- note added: "10K Pot"
- note added: "FIXED GAIN\nAv=13.5 \n(+22.61dB)"
- note added: "OPA227P"
- note added: "OUTPUT"
- note added: "RB1/RB2 tuned \nfor 10K Pot\n"
- note added: "VAR GAIN\nAv=6.3\n(+16dB)"
- note added: "VAR OFFSET"
- note removed: "10K POT\n"

Commit message: Board Layout completed
Parts:
- added J_OUT1: Conn_01x02, Connector_PinSocket_2.54mm:PinSocket_1x02_P2.54mm_Vertical, symbol Connector_Generic:Conn_01x02
- C1: renamed from C?; value CP -> 330nF; footprint (none) -> Capacitor_THT:C_Rect_L7.2mm_W2.5mm_P5.00mm_FKS2_FKP2_MKS2_MKP2
- C2: renamed from C?; value CP -> 100nF; footprint (none) -> Capacitor_THT:C_Rect_L7.2mm_W2.5mm_P5.00mm_FKS2_FKP2_MKS2_MKP2
- J_AD9833: footprint (none) -> Connector_PinSocket_2.54mm:PinSocket_1x07_P2.54mm_Vertical
- J_AMP1, J_FREQ1, J_FREQ2, J_OFFSET1, J_PWR1, J_VEL1: footprint (none) -> Connector_PinSocket_2.54mm:PinSocket_1x03_P2.54mm_Vertical
- J_OLED1: footprint (none) -> Connector_PinSocket_2.54mm:PinSocket_1x04_P2.54mm_Vertical
- J_TX1: footprint (none) -> Connector_PinSocket_2.54mm:PinSocket_1x15_P2.54mm_Vertical
- J_VIN1: renamed from J_VIN; footprint (none) -> Connector_PinSocket_2.54mm:PinSocket_1x15_P2.54mm_Vertical
- RB1, RB2, R_AF1, R_AG1, R_AMP1, R_AMP2, R_FUNC1, R_MIX1, R_MIX2, R_MODE1, R_VEL1: footprint (none) -> Resistor_THT:R_Axial_DIN0207_L6.3mm_D2.5mm_P7.62mm_Horizontal
- SW_FUNC1, SW_MODE1: footprint (none) -> Button_Switch_THT:SW_PUSH_6mm
- U2: renamed from U?; footprint (none) -> Package_DIP:DIP-8_W7.62mm_Socket
- U_OUTPUT1: footprint (none) -> Package_DIP:DIP-8_W7.62mm_Socket
- gave numbers to parts that had none: 1
Connections:
- net labels removed: POT_CS
- wire segments 116 -> 118
- no-connect marks 1 -> 17

Commit message: changed to SMT. Added proper spaces for pots
Parts:
- C1, C2: footprint Capacitor_THT:C_Rect_L7.2mm_W2.5mm_P5.00mm_FKS2_FKP2_MKS2_MKP2 -> Capacitor_SMD:C_0805_2012Metric_Pad1.15x1.40mm_HandSolder
- RB1, RB2, R_AF1, R_AG1, R_AMP1, R_AMP2, R_FUNC1, R_MIX1, R_MIX2, R_MODE1, R_VEL1: footprint Resistor_THT:R_Axial_DIN0207_L6.3mm_D2.5mm_P7.62mm_Horizontal -> Resistor_SMD:R_0805_2012Metric_Pad1.15x1.40mm_HandSolder
- U2, U_OUTPUT1: footprint Package_DIP:DIP-8_W7.62mm_Socket -> Package_SO:SOIC-8_3.9x4.9mm_P1.27mm
Changed lines of the file:
@@
 F 0 "C1" H 2575 1900 50  0000 L CNN
 F 1 "330nF" H 2575 1700 50  0000 L CNN
-F 2 "Capacitor_THT:C_Rect_L7.2mm_W2.5mm_P5.00mm_FKS2_FKP2_MKS2_MKP2" H 2588 1650 50  0001 C CNN
+F 2 "Capacitor_SMD:C_0805_2012Metric_Pad1.15x1.40mm_HandSolder" H 2588 1650 50  0001 C CNN
 F 3 "" H 2550 1800 50  0001 C CNN
 	1    2550 1800
@@
 F 0 "C2" H 3675 1900 50  0000 L CNN
 F 1 "100nF" H 3675 1700 50  0000 L CNN
-F 2 "Capacitor_THT:C_Rect_L7.2mm_W2.5mm_P5.00mm_FKS2_FKP2_MKS2_MKP2" H 3688 1650 50  0001 C CNN
+F 2 "Capacitor_SMD:C_0805_2012Metric_Pad1.15x1.40mm_HandSolder" H 3688 1650 50  0001 C CNN
 F 3 "" H 3650 1800 50  0001 C CNN
 	1    3650 1800
@@
 F 0 "R_MODE1" V 2096 6650 50  0000 C CNN
 F 1 "1K" V 2185 6650 50  0000 C CNN
-F 2 "Resistor_THT:R_Axial_DIN0207_L6.3mm_D2.5mm_P7.62mm_Horizontal" V 2230 6650 50  0001 C CNN
+F 2 "Resistor_SMD:R_0805_2012Metric_Pad1.15x1.40mm_HandSolder" V 2230 6650 50  0001 C CNN
 F 3 "~" H 2300 6650 50  0001 C CNN
 	1    2300 6650
@@
 F 0 "R_FUNC1" V 2096 7050 50  0000 C CNN
 F 1 "1K" V 2185 7050 50  0000 C CNN
-F 2 "Resistor_THT:R_Axial_DIN0207_L6.3mm_D2.5mm_P7.62mm_Horizontal" V 2230 7050 50  0001 C CNN
+F 2 "Resistor_SMD:R_0805_2012Metric_Pad1.15x1.40mm_HandSolder" V 2230 7050 50  0001 C CNN
 F 3 "~" H 2300 7050 50  0001 C CNN
 	1    2300 7050
@@
 F 0 "R_VEL1" V 7850 5775 50  0000 C CNN
 F 1 "1K" V 7750 5775 50  0000 C CNN
-F 2 "Resistor_THT:R_Axial_DIN0207_L6.3mm_D2.5mm_P7.62mm_Horizontal" V 7680 5775 50  0001 C CNN
+F 2 "Resistor_SMD:R_0805_2012Metric_Pad1.15x1.40mm_HandSolder" V 7680 5775 50  0001 C CNN
 F 3 "~" H 7750 5775 50  0001 C CNN
 	1    7750 5775
@@
 F 0 "R_AG1" H 6870 3795 50  0000 L CNN
 F 1 "1K2" H 6870 3706 50  0000 L CNN
-F 2 "Resistor_THT:R_Axial_DIN0207_L6.3mm_D2.5mm_P7.62mm_Horizontal" V 6730 3750 50  0001 C CNN
+F 2 "Resistor_SMD:R_0805_2012Metric_Pad1.15x1.40mm_HandSolder" V 6730 3750 50  0001 C CNN
 F 3 "~" H 6800 3750 50  0001 C CNN
 	1    6800 3750
@@
 F 0 "R_MIX2" H 8430 2255 50  0000 R CNN
 F 1 "1K" H 8430 2344 50  0000 R CNN
-F 2 "Resistor_THT:R_Axial_DIN0207_L6.3mm_D2.5mm_P7.62mm_Horizontal" V 8430 2300 50  0001 C CNN
+F 2 "Resistor_SMD:R_0805_2012Metric_Pad1.15x1.40mm_HandSolder" V 8430 2300 50  0001 C CNN
 F 3 "~" H 8500 2300 50  0001 C CNN
 	1    8500 2300
@@
 F 0 "R_MIX1" H 8430 2655 50  0000 R CNN
 F 1 "1K" H 8430 2744 50  0000 R CNN
-F 2 "Resistor_THT:R_Axial_DIN0207_L6.3mm_D2.5mm_P7.62mm_Horizontal" V 8430 2700 50  0001 C CNN
+F 2 "Resistor_SMD:R_0805_2012Metric_Pad1.15x1.40mm_HandSolder" V 8430 2700 50  0001 C CNN
 F 3 "~" H 8500 2700 50  0001 C CNN
 	1    8500 2700
@@
 F 0 "RB2" H 6620 2245 50  0000 L CNN
 F 1 "1K" H 6620 2156 50  0000 L CNN
-F 2 "Resistor_THT:R_Axial_DIN0207_L6.3mm_D2.5mm_P7.62mm_Horizontal" V 6480 2200 50  0001 C CNN
+F 2 "Resistor_SMD:R_0805_2012Metric_Pad1.15x1.40mm_HandSolder" V 6480 2200 50  0001 C CNN
 F 3 "~" H 6550 2200 50  0001 C CNN
 	1    6550 2200
@@
 F 0 "R_AF1" V 7400 3550 50  0000 C CNN
 F 1 "15K" V 7500 3550 50  0000 C CNN
-F 2 "Resistor_THT:R_Axial_DIN0207_L6.3mm_D2.5mm_P7.62mm_Horizontal" V 7230 3550 50  0001 C CNN
+F 2 "Resistor_SMD:R_0805_2012Metric_Pad1.15x1.40mm_HandSolder" V 7230 3550 50  0001 C CNN
 F 3 "~" H 7300 3550 50  0001 C CNN
 	1    7300 3550
@@
 F 0 "RB1" H 6620 1545 50  0000 L CNN
 F 1 "8K2" H 6620 1456 50  0000 L CNN
-F 2 "Resistor_THT:R_Axial_DIN0207_L6.3mm_D2.5mm_P7.62mm_Horizontal" V 6480 1500 50  0001 C CNN
+F 2 "Resistor_SMD:R_0805_2012Metric_Pad1.15x1.40mm_HandSolder" V 6480 1500 50  0001 C CNN
 F 3 "~" H 6550 1500 50  0001 C CNN
 	1    6550 1500
@@
 F 0 "U_OUTPUT1" H 9600 2750 50  0000 L CNN
 F 1 "OPA1641" H 9600 2850 50  0000 L CNN
-F 2 "Package_DIP:DIP-8_W7.62mm_Socket" H 9500 2600 50  0001 C CNN
+F 2 "Package_SO:SOIC-8_3.9x4.9mm_P1.27mm" H 9500 2600 50  0001 C CNN
 F 3 "http://www.ti.com/lit/ds/symlink/opa1641.pdf" H 9500 2600 50  0001 C CNN
 	1    9500 2600
@@
 F 0 "R_AMP1" H 8600 3700 50  0000 L CNN
 F 1 "1K8" H 8650 3600 50  0000 L CNN
-F 2 "Resistor_THT:R_Axial_DIN0207_L6.3mm_D2.5mm_P7.62mm_Horizontal" V 8830 3650 50  0001 C CNN
+F 2 "Resistor_SMD:R_0805_2012Metric_Pad1.15x1.40mm_HandSolder" V 8830 3650 50  0001 C CNN
 F 3 "~" H 8900 3650 50  0001 C CNN
 	1    8900 3650
@@
 F 0 "R_AMP2" H 8550 4100 50  0000 L CNN
 F 1 "470R" H 8650 4000 50  0000 L CNN
-F 2 "Resistor_THT:R_Axial_DIN0207_L6.3mm_D2.5mm_P7.62mm_Horizontal" V 8830 4050 50  0001 C CNN
+F 2 "Resistor_SMD:R_0805_2012Metric_Pad1.15x1.40mm_HandSolder" V 8830 4050 50  0001 C CNN
 F 3 "~" H 8900 4050 50  0001 C CNN
 	1    8900 4050
@@
 F 0 "U2" H 7790 1995 50  0000 L CNN
 F 1 "TL072" H 7790 1906 50  0000 L CNN
-F 2 "Package_DIP:DIP-8_W7.62mm_Socket" H 7450 1950 50  0001 C CNN
+F 2 "Package_SO:SOIC-8_3.9x4.9mm_P1.27mm" H 7450 1950 50  0001 C CNN
 F 3 "" H 7450 1950 50  0001 C CNN
 	2    7450 1950
@@
 F 0 "U2" H 7590 3045 50  0000 L CNN
 F 1 "TL072" H 7590 2956 50  0000 L CNN
-F 2 "Package_DIP:DIP-8_W7.62mm_Socket" H 7250 3000 50  0001 C CNN
+F 2 "Package_SO:SOIC-8_3.9x4.9mm_P1.27mm" H 7250 3000 50  0001 C CNN
 F 3 "" H 7250 3000 50  0001 C CNN
 	1    7250 3000

Commit message: Changed to 4 layer board. Middle layers for 5V and GND. Signal traces on top layer, +/-12V and HF digital signals on bottom layer
Parts:
- added C_BP1, C_BP2, C_BP3, C_BP4: 100nF, Capacitor_SMD:C_0805_2012Metric_Pad1.15x1.40mm_HandSolder, symbol Device:C
Connections:
- wire segments 118 -> 133
