File: Hardware/AD9833FunctionGenerator.sch (KiCad schematic (older format))
At the start: 33 parts, among them U1 LM7805_TO220, U2 TL072

Commit message: updated hardware
- changed output opamp to inverting to allow 0V-20Vpp output
Parts:
- removed R_AMP2: 470R, Resistor_SMD:R_0805_2012Metric_Pad1.15x1.40mm_HandSolder, symbol Device:R
- removed U2: TL072, Package_SO:SOIC-8_3.9x4.9mm_P1.27mm, symbol AD9833FunctionGenerator-rescue:TL072
- removed U_OUTPUT1: OPA1641, Package_SO:SOIC-8_3.9x4.9mm_P1.27mm, symbol Amplifier_Operational:OPA1641
- added C_OUT1: 10nF, Capacitor_SMD:C_0805_2012Metric_Pad1.15x1.40mm_HandSolder, symbol Device:C
- added U_AMP1, U_COMP1: TL072, Package_SO:SOIC-8_3.9x4.9mm_P1.27mm, symbol Amplifier_Operational:TL072
- R_AMP1: value 1K8 -> 1K5
Connections:
- net labels removed: OUTPUT
- wire segments 133 -> 134
- no-connect marks 17 -> 20
Other:
- note added: "RB1/RB2 \ntuned for\n10K Pot\n"
- note added: "VAR GAIN\nAv=-6.3\n(+16dB)"
- note removed: "Direct Digital Synthesis Molex socket"
- note removed: "OLED Display Molex socket"
- note removed: "OPA227P"
- note removed: "Potentiometer Molex Sockets"
- note removed: "RB1/RB2 tuned \nfor 10K Pot\n"
- note removed: "SPST Molex Sockets"
- note removed: "VAR GAIN\nAv=6.3\n(+16dB)"

Commit message: Changed J_PWR1 from 01x03 to 02x05
Parts:
- removed J_PWR1: Conn_01x03, Connector_PinSocket_2.54mm:PinSocket_1x03_P2.54mm_Vertical, symbol Connector_Generic:Conn_01x03
- added J_PWR1: Conn_02x05_Odd_Even, Connector_PinHeader_2.54mm:PinHeader_2x05_P2.54mm_Vertical, symbol Connector_Generic:Conn_02x05_Odd_Even
Connections:
- wire segments 134 -> 144
Changed lines of the file:
@@
 $EndComp
 Wire Wire Line
-	1500 1750 1800 1750
-Text Label 1550 1750 0    50   ~ 0
+	1950 1800 2200 1800
+Text Label 2000 1800 0    50   ~ 0
 GND
 Wire Wire Line
@@
 L Device:CP C1
 U 1 1 5B8B3473
-P 2550 1800
-F 0 "C1" H 2575 1900 50  0000 L CNN
-F 1 "330nF" H 2575 1700 50  0000 L CNN
-F 2 "Capacitor_SMD:C_0805_2012Metric_Pad1.15x1.40mm_HandSolder" H 2588 1650 50  0001 C CNN
-F 3 "" H 2550 1800 50  0001 C CNN
-	1    2550 1800
+P 2800 1800
+F 0 "C1" H 2825 1900 50  0000 L CNN
+F 1 "330nF" H 2825 1700 50  0000 L CNN
+F 2 "Capacitor_SMD:C_0805_2012Metric_Pad1.15x1.40mm_HandSolder" H 2838 1650 50  0001 C CNN
+F 3 "" H 2800 1800 50  0001 C CNN
+	1    2800 1800
 	1    0    0    -1
 $EndComp
@@
 L Device:CP C2
 U 1 1 5B8B34AC
-P 3650 1800
-F 0 "C2" H 3675 1900 50  0000 L CNN
-F 1 "100nF" H 3675 1700 50  0000 L CNN
-F 2 "Capacitor_SMD:C_0805_2012Metric_Pad1.15x1.40mm_HandSolder" H 3688 1650 50  0001 C CNN
-F 3 "" H 3650 1800 50  0001 C CNN
-	1    3650 1800
-	1    0    0    -1
-$EndComp
-Wire Wire Line
-	2550 1450 2550 1650
-Wire Wire Line
-	3350 1450 3650 1450
-Wire Wire Line
-	3650 1450 3650 1650
-Wire Wire Line
-	3050 1750 3050 2050
-Wire Wire Line
-	2550 1950 2550 2050
-Wire Wire Line
-	2550 2050 3050 2050
-Connection ~ 3050 2050
-Wire Wire Line
-	3650 2050 3650 1950
-Text Label 3050 2350 1    50   ~ 0
-GND
-Text Label 1750 1650 2    50   ~ 0
+P 3900 1800
+F 0 "C2" H 3925 1900 50  0000 L CNN
+F 1 "100nF" H 3925 1700 50  0000 L CNN
+F 2 "Capacitor_SMD:C_0805_2012Metric_Pad1.15x1.40mm_HandSolder" H 3938 1650 50  0001 C CNN
+F 3 "" H 3900 1800 50  0001 C CNN
+	1    3900 1800
+	1    0    0    -1
+$EndComp
+Wire Wire Line
+	2800 1450 2800 1650
+Wire Wire Line
+	3600 1450 3900 1450
+Wire Wire Line
+	3900 1450 3900 1650
+Wire Wire Line
+	3300 1750 3300 2050
+Wire Wire Line
+	2800 1950 2800 2050
+Wire Wire Line
+	2800 2050 3300 2050
+Connection ~ 3300 2050
+Wire Wire Line
+	3900 2050 3900 1950
+Text Label 3300 2350 1    50   ~ 0
+GND
+Text Label 2150 1600 2    50   ~ 0
 +12V
-Connection ~ 3650 1450
-Text Label 3950 1450 2    50   ~ 0
+Connection ~ 3900 1450
+Text Label 4200 1450 2    50   ~ 0
 5V
 $Comp
@@
 SIGFUNC
 Wire Wire Line
-	2550 1450 2750 1450
-Wire Wire Line
-	3050 2050 3050 2350
-Wire Wire Line
-	3050 2050 3650 2050
-Wire Wire Line
-	3650 1450 3950 1450
+	2800 1450 3000 1450
+Wire Wire Line
+	3300 2050 3300 2350
+Wire Wire Line
+	3300 2050 3900 2050
+Wire Wire Line
+	3900 1450 4200 1450
 $Comp
 L Regulator_Linear:LM7805_TO220 U1
 U 1 1 5BA958E1
-P 3050 1450
-F 0 "U1" H 3050 1689 50  0000 C CNN
-F 1 "LM7805_TO220" H 3050 1600 50  0000 C CNN
-F 2 "Package_TO_SOT_THT:TO-220-3_Vertical" H 3050 1675 50  0001 C CIN
-F 3 "http://www.fairchildsemi.com/ds/LM/LM7805.pdf" H 3050 1400 50  0001 C CNN
-	1    3050 1450
+P 3300 1450
+F 0 "U1" H 3300 1689 50  0000 C CNN
+F 1 "LM7805_TO220" H 3300 1600 50  0000 C CNN
+F 2 "Package_TO_SOT_THT:TO-220-3_Vertical" H 3300 1675 50  0001 C CIN
+F 3 "http://www.fairchildsemi.com/ds/LM/LM7805.pdf" H 3300 1400 50  0001 C CNN
+	1    3300 1450
 	1    0    0    -1
 $EndComp
@@
 Wire Wire Line
 	3525 4600 3300 4600
-$Comp
-L Connector_Generic:Conn_01x03 J_PWR1
-U 1 1 5BB5F964
-P 1300 1750
-F 0 "J_PWR1" H 1200 2000 50  0000 C CNN
-F 1 "Conn_01x03" H 1100 2000 50  0001 C CNN
-F 2 "Connector_PinSocket_2.54mm:PinSocket_1x03_P2.54mm_Vertical" H 1300 1750 50  0001 C CNN
-F 3 "~" H 1300 1750 50  0001 C CNN
-	1    1300 1750
-	-1   0    0    -1
-$EndComp
-Wire Wire Line
-	1500 1850 1800 1850
-Text Label 1700 1850 2    50   ~ 0
+Wire Wire Line
+	1850 2000 2200 2000
+Text Label 2150 2000 2    50   ~ 0
 -12V
 Wire Wire Line
@@
 L power:PWR_FLAG #FLG0101
 U 1 1 5BB589B5
-P 1800 1650
-F 0 "#FLG0101" H 1800 1725 50  0001 C CNN
-F 1 "PWR_FLAG" V 1800 1800 50  0001 L CNN
-F 2 "" H 1800 1650 50  0001 C CNN
-F 3 "~" H 1800 1650 50  0001 C CNN
-	1    1800 1650
+P 2200 1600
+F 0 "#FLG0101" H 2200 1675 50  0001 C CNN
+F 1 "PWR_FLAG" V 2200 1750 50  0001 L CNN
+F 2 "" H 2200 1600 50  0001 C CNN
+F 3 "~" H 2200 1600 50  0001 C CNN
+	1    2200 1600
 	0    1    1    0
 $EndComp
@@
 L power:PWR_FLAG #FLG0102
 U 1 1 5BB5C39F
-P 1800 1750
-F 0 "#FLG0102" H 1800 1825 50  0001 C CNN
-F 1 "PWR_FLAG" V 1800 1900 50  0001 L CNN
-F 2 "" H 1800 1750 50  0001 C CNN
-F 3 "~" H 1800 1750 50  0001 C CNN
-	1    1800 1750
-	0    1    1    0
-$EndComp
-Wire Wire Line
-	1500 1650 1800 1650
+P 2200 1800
+F 0 "#FLG0102" H 2200 1875 50  0001 C CNN
+F 1 "PWR_FLAG" V 2200 1950 50  0001 L CNN
+F 2 "" H 2200 1800 50  0001 C CNN
+F 3 "~" H 2200 1800 50  0001 C CNN
+	1    2200 1800
+	0    1    1    0
+$EndComp
+Wire Wire Line
+	1850 1600 2200 1600
 $Comp
 L power:PWR_FLAG #FLG0103
 U 1 1 5BB669DD
-P 1800 1850
-F 0 "#FLG0103" H 1800 1925 50  0001 C CNN
-F 1 "PWR_FLAG" V 1800 2000 50  0001 L CNN
-F 2 "" H 1800 1850 50  0001 C CNN
-F 3 "~" H 1800 1850 50  0001 C CNN
-	1    1800 1850
-	0    1    1    0
-$EndComp
-Wire Wire Line
-	2550 1450 2250 1450
-Connection ~ 2550 1450
-Text Label 2250 1450 0    50   ~ 0
+P 2200 2000
+F 0 "#FLG0103" H 2200 2075 50  0001 C CNN
+F 1 "PWR_FLAG" V 2200 2150 50  0001 L CNN
+F 2 "" H 2200 2000 50  0001 C CNN
+F 3 "~" H 2200 2000 50  0001 C CNN
+	1    2200 2000
+	0    1    1    0
+$EndComp
+Wire Wire Line
+	2800 1450 2500 1450
+Connection ~ 2800 1450
+Text Label 2500 1450 0    50   ~ 0
 +12V
 $Comp
@@
 Wire Wire Line
 	6200 1500 6150 1500
+Wire Wire Line
+	1950 1800 1950 1700
+Wire Wire Line
+	1950 1700 1850 1700
+Wire Wire Line
+	1950 1800 1950 1900
+Wire Wire Line
+	1950 1900 1850 1900
+Connection ~ 1950 1800
+Wire Wire Line
+	1950 1800 1850 1800
+$Comp
+L Connector_Generic:Conn_02x05_Odd_Even J_PWR1
+U 1 1 5BBA34EF
+P 1550 1800
+F 0 "J_PWR1" H 1600 2217 50  0000 C CNN
+F 1 "Conn_02x05_Odd_Even" H 1600 2126 50  0000 C CNN
+F 2 "Connector_PinHeader_2.54mm:PinHeader_2x05_P2.54mm_Vertical" H 1550 1800 50  0001 C CNN
+F 3 "~" H 1550 1800 50  0001 C CNN
+	1    1550 1800
+	1    0    0    -1
+$EndComp
+Wire Wire Line
+	1350 1600 1100 1600
+Wire Wire Line
+	1350 1700 1100 1700
+Wire Wire Line
+	1100 1800 1350 1800
+Wire Wire Line
+	1100 1900 1350 1900
+Wire Wire Line
+	1100 2000 1350 2000
+Text Label 1100 1600 0    50   ~ 0
++12V
+Text Label 1100 1700 0    50   ~ 0
+GND
+Text Label 1100 1800 0    50   ~ 0
+GND
+Text Label 1100 1900 0    50   ~ 0
+GND
+Text Label 1100 2000 0    50   ~ 0
+-12V
 $EndSCHEMATC

Commit message: added MCP42050
Parts:
- removed C_OUT1: 10nF, Capacitor_SMD:C_0805_2012Metric_Pad1.15x1.40mm_HandSolder, symbol Device:C
- removed R_AF1: 15K, Resistor_SMD:R_0805_2012Metric_Pad1.15x1.40mm_HandSolder, symbol Device:R
- removed R_AG1: 1K2, Resistor_SMD:R_0805_2012Metric_Pad1.15x1.40mm_HandSolder, symbol Device:R
- removed R_AMP1: 1K5, Resistor_SMD:R_0805_2012Metric_Pad1.15x1.40mm_HandSolder, symbol Device:R
- removed unit 1 of U_COMP1
- added R_1: 1K, symbol Device:R
- added R_RANGE1: 1K, Resistor_SMD:R_0805_2012Metric_Pad1.15x1.40mm_HandSolder, symbol Device:R
- added SW_RANGE1: SW_SPST, Button_Switch_THT:SW_PUSH_6mm, symbol Switch:SW_SPST
- added U?: MCP42050, symbol Potentiometer_Digital:MCP42050
- renumbered U_COMP1 to U_OUT1, U_AMP1 to U_OUT1
Connections:
- net labels added: FUNCMODE1, FUNCSIG, POT_CS, RANGEMODE1, RANGE_RELAY_EN, SWEEPMODE1
- net labels removed: FUNC1, MODE1, SIGFUNC
- wire segments 144 -> 158
- no-connect marks 20 -> 18
Other:
- note removed: "FIXED GAIN\nAv=13.5 \n(+22.61dB)"
- note removed: "VAR GAIN\nAv=-6.3\n(+16dB)"

Commit message: update
Parts:
- removed C_BP1, C_BP2, C_BP3, C_BP4: 100nF, Capacitor_SMD:C_0805_2012Metric_Pad1.15x1.40mm_HandSolder, symbol Device:C
- removed U_AMP1, U_COMP1, U_OUT1 (x2): TL072, Package_SO:SOIC-8_3.9x4.9mm_P1.27mm, symbol Amplifier_Operational:TL072
- added R?: 1K, symbol Device:R
- added U? (x3): TL071, symbol Amplifier_Operational:TL071
- RB1: value 8K2 -> 1K
- R_1, R_MIX1, R_MIX2: value 1K -> 10K
Connections:
- wire segments 158 -> 150
- no-connect marks 18 -> 24
Other:
- note added: "10K"
- note added: "BUFFER"
- note added: "GAIN"
- note added: "MIXER"
- note added: "adjust \nRB1/RB2 \nfor center \noffset"
- note removed: "RB1/RB2 \ntuned for\n10K Pot\n"
- note removed: "VAR OFFSET"

Commit message: updated SW and HW
- Added LM7171 output sectionz. 20Vp-p output, +26db gain, no cutoff up to 100KHz.
- Corrected output section offset controls
- Added phase control code (not working)
Parts:
- added CF1: 10pF, symbol Device:C
- added R_ISO1: 330R, symbol Device:R
- R1: renamed from R?; value 1K -> 1K5
- RB1: value 1K -> 147K
- RB2: value 1K -> 82K
- R_VEL1: value 1K -> 100R
- gave numbers to parts that had none: 4
- renumbered R_1 to RF1
Connections:
- net labels removed: RANGE_RELAY_EN
- wire segments 150 -> 157
- no-connect marks 24 -> 25
Other:
- note added: "B50K"
- note added: "LM7171"
- note removed: "10K"
Changed lines of the file:
@@
 P 6600 7075
 F 0 "R_VEL1" V 6700 7075 50  0000 C CNN
-F 1 "1K" V 6600 7075 50  0000 C CNN
+F 1 "100R" V 6600 7075 50  0000 C CNN
 F 2 "Resistor_SMD:R_0805_2012Metric_Pad1.15x1.40mm_HandSolder" V 6530 7075 50  0001 C CNN
 F 3 "~" H 6600 7075 50  0001 C CNN
@@
 U 1 1 5BB26E72
 P 5400 1700
-F 0 "J_OFFSET1" H 5300 1450 50  0000 C CNN
+F 0 "J_OFFSET1" H 5700 1650 50  0000 C CNN
 F 1 "Conn_01x03" H 5450 1350 50  0001 C CNN
 F 2 "Connector_PinSocket_2.54mm:PinSocket_1x03_P2.54mm_Vertical" H 5400 1700 50  0001 C CNN
@@
 P 5800 1800
 F 0 "RB2" V 5900 1750 50  0000 L CNN
-F 1 "1K" V 5800 1750 50  0000 L CNN
+F 1 "82K" V 5800 1750 50  0000 L CNN
 F 2 "Resistor_SMD:R_0805_2012Metric_Pad1.15x1.40mm_HandSolder" V 5730 1800 50  0001 C CNN
 F 3 "~" H 5800 1800 50  0001 C CNN
@@
 P 5800 1600
 F 0 "RB1" V 5700 1550 50  0000 L CNN
-F 1 "1K" V 5800 1550 50  0000 L CNN
+F 1 "147K" V 5800 1500 50  0000 L CNN
 F 2 "Resistor_SMD:R_0805_2012Metric_Pad1.15x1.40mm_HandSolder" V 5730 1600 50  0001 C CNN
 F 3 "~" H 5800 1600 50  0001 C CNN
@@
 L Connector_Generic:Conn_01x02 J_OUT1
 U 1 1 5BB86F40
-P 9800 2200
-F 0 "J_OUT1" H 9650 2350 50  0000 L CNN
-F 1 "Conn_01x02" H 9880 2101 50  0001 L CNN
-F 2 "Connector_PinSocket_2.54mm:PinSocket_1x02_P2.54mm_Vertical" H 9800 2200 50  0001 C CNN
-F 3 "~" H 9800 2200 50  0001 C CNN
-	1    9800 2200
-	1    0    0    -1
-$EndComp
-Wire Wire Line
-	9600 2300 9550 2300
-Text Label 9550 2400 3    50   ~ 0
+P 10350 2200
+F 0 "J_OUT1" H 10200 2350 50  0000 L CNN
+F 1 "Conn_01x02" H 10430 2101 50  0001 L CNN
+F 2 "Connector_PinSocket_2.54mm:PinSocket_1x02_P2.54mm_Vertical" H 10350 2200 50  0001 C CNN
+F 3 "~" H 10350 2200 50  0001 C CNN
+	1    10350 2200
+	1    0    0    -1
+$EndComp
+Wire Wire Line
+	10150 2300 10100 2300
+Text Label 10100 2400 3    50   ~ 0
 GND
 Wire Wire Line
@@
 $EndComp
 Wire Wire Line
-	1350 1600 1100 1600
-Wire Wire Line
-	1350 1700 1100 1700
-Wire Wire Line
-	1100 1800 1350 1800
-Wire Wire Line
-	1100 1900 1350 1900
-Wire Wire Line
-	1100 2000 1350 2000
-Text Label 1100 1600 0    50   ~ 0
+	1350 1600 1050 1600
+Wire Wire Line
+	1350 1700 1250 1700
+Wire Wire Line
+	1050 1800 1250 1800
+Wire Wire Line
+	1250 1900 1350 1900
+Wire Wire Line
+	1050 2000 1350 2000
+Text Label 1050 1600 0    50   ~ 0
 +12V
-Text Label 1100 1700 0    50   ~ 0
+Text Label 1050 1800 0    50   ~ 0
 GND
-Text Label 1100 1800 0    50   ~ 0
-GND
-Text Label 1100 1900 0    50   ~ 0
-GND
-Text Label 1100 2000 0    50   ~ 0
+Text Label 1050 2000 0    50   ~ 0
 -12V
 Wire Wire Line
 	1900 4000 1250 4000
-Wire Wire Line
-	1900 4100 1250 4100
-Text Label 1250 4100 0    50   ~ 0
-RANGE_RELAY_EN
 $Comp
 L Switch:SW_SPST SW_RANGE1
@@
 	5650 4450 5300 4450
 $Comp
-L Potentiometer_Digital:MCP42050 U?
+L Potentiometer_Digital:MCP42050 U2
 U 1 1 5BB5DA86
 P 6150 4750
-F 0 "U?" H 5750 5400 50  0000 C CNN
+F 0 "U2" H 5750 5400 50  0000 C CNN
 F 1 "MCP42050" H 5750 5300 50  0000 C CNN
 F 2 "" H 6150 4850 50  0001 C CNN
@@
 	5200 3000 5600 3000
 $Comp
-L Device:R R_1
+L Device:R RF1
 U 1 1 5BCBCF93
 P 7350 3100
-F 0 "R_1" V 7450 3100 50  0000 C CNN
+F 0 "RF1" V 7450 3100 50  0000 C CNN
 F 1 "10K" V 7350 3100 50  0000 C CNN
 F 2 "" V 7280 3100 50  0001 C CNN
@@
 	6900 2400 7050 2400
 $Comp
-L Amplifier_Operational:TL071 U?
+L Amplifier_Operational:TL071 U_GAIN1
 U 1 1 5BB7F23F
 P 8800 2200
-F 0 "U?" H 8900 2450 50  0000 L CNN
+F 0 "U_GAIN1" H 8900 2450 50  0000 L CNN
 F 1 "TL071" H 8900 2500 50  0000 L CNN
 F 2 "" H 8850 2250 50  0001 C CNN
@@
 $EndComp
 $Comp
-L Amplifier_Operational:TL071 U?
+L Amplifier_Operational:TL071 U_BUFF1
 U 1 1 5BB7F589
 P 5900 3100
-F 0 "U?" H 5950 3300 50  0000 L CNN
+F 0 "U_BUFF1" H 5950 3300 50  0000 L CNN
 F 1 "TL071" H 5950 3350 50  0000 L CNN
 F 2 "" H 5950 3150 50  0001 C CNN
@@
 	6000 1800 5950 1800
 Wire Wire Line
-	9550 2300 9550 2400
-$Comp
-L Amplifier_Operational:TL071 U?
+	10100 2300 10100 2400
+$Comp
+L Amplifier_Operational:TL071 U_MIX1
 U 1 1 5BB7F607
 P 7350 2300
-F 0 "U?" H 7400 2550 50  0000 L CNN
+F 0 "U_MIX1" H 7400 2550 50  0000 L CNN
 F 1 "TL071" H 7400 2600 50  0000 L CNN
 F 2 "" H 7400 2350 50  0001 C CNN
@@
 	6400 2400 6900 2400
 $Comp
-L Device:R R?
+L Device:R R1
 U 1 1 5BDB0D4B
 P 8150 2300
-F 0 "R?" V 8250 2300 50  0000 C CNN
-F 1 "1K" V 8150 2300 50  0000 C CNN
+F 0 "R1" V 8250 2300 50  0000 C CNN
+F 1 "1K5" V 8150 2300 50  0000 C CNN
 F 2 "" V 8080 2300 50  0001 C CNN
 F 3 "~" H 8150 2300 50  0001 C CNN
@@
 Wire Wire Line
 	8950 2900 9200 2900
-Wire Wire Line
-	9600 2200 9200 2200
-Connection ~ 9200 2200
 Text Notes 8800 3650 0    50   ~ 0
-10K
+B50K
 Text Notes 8800 2700 0    50   ~ 0
 GAIN
@@
 Text Notes 5900 3550 0    50   ~ 0
 BUFFER
+$Comp
+L Device:R R_ISO1
+U 1 1 5BB84CB7
+P 9550 2200
+F 0 "R_ISO1" V 9346 2200 50  0000 C CNN
+F 1 "330R" V 9435 2200 50  0000 C CNN
+F 2 "" V 9480 2200 50  0001 C CNN
+F 3 "~" H 9550 2200 50  0001 C CNN
+	1    9550 2200
+	0    1    1    0
+$EndComp
+Wire Wire Line
+	9200 2200 9400 2200
+Connection ~ 9200 2200
+Wire Wire Line
+	9700 2200 10150 2200
+Text Notes 8900 1850 0    50   ~ 0
+LM7171
+Text Notes 7400 1950 0    50   ~ 0
+LM7171
+$Comp
+L Device:C CF1
+U 1 1 5BB9124E
+P 8850 4000
+F 0 "CF1" V 8601 4000 50  0000 C CNN
+F 1 "10pF" V 8690 4000 50  0000 C CNN
+F 2 "" H 8888 3850 50  0001 C CNN
+F 3 "~" H 8850 4000 50  0001 C CNN
+	1    8850 4000
+	0    1    1    0
+$EndComp
+Wire Wire Line
+	8700 4000 8400 4000
+Wire Wire Line
+	8400 4000 8400 2900
+Connection ~ 8400 2900
+Wire Wire Line
+	9000 4000 9200 4000
+Wire Wire Line
+	9200 4000 9200 2900
+Connection ~ 9200 2900
+NoConn ~ 1900 4100
+Text Notes 5050 1800 0    50   ~ 0
+B50K
+Wire Wire Line
+	1250 1700 1250 1800
+Connection ~ 1250 1800
+Wire Wire Line
+	1250 1800 1350 1800
+Wire Wire Line
+	1250 1800 1250 1900
 $EndSCHEMATC

Commit message: updated HW
- Changed Offset and Amp pots from 50K to 10: (better part availability)
- Adjusted opamp gain resistors ratio
- Added 100K trim pots for eaiser offset center adjustment
Parts:
- removed RB1: 147K, Resistor_SMD:R_0805_2012Metric_Pad1.15x1.40mm_HandSolder, symbol Device:R
- removed RB2: 82K, Resistor_SMD:R_0805_2012Metric_Pad1.15x1.40mm_HandSolder, symbol Device:R
- added OFF1, OFF2: 100K, symbol Device:R_POT_TRIM
- CF1: value 10pF -> 2pF
- R1: value 1K5 -> 390R
Connections:
- wire segments 157 -> 165
Other:
- note added: "B10K"
- note removed: "B50K"
- note removed: "adjust \nRB1/RB2 \nfor center \noffset"
Changed lines of the file:
@@
 	-1   0    0    1
 $EndComp
-$Comp
-L Device:R RB2
-U 1 1 5BB2B576
-P 5800 1800
-F 0 "RB2" V 5900 1750 50  0000 L CNN
-F 1 "82K" V 5800 1750 50  0000 L CNN
-F 2 "Resistor_SMD:R_0805_2012Metric_Pad1.15x1.40mm_HandSolder" V 5730 1800 50  0001 C CNN
-F 3 "~" H 5800 1800 50  0001 C CNN
-	1    5800 1800
-	0    1    1    0
-$EndComp
-Wire Wire Line
-	5600 1800 5650 1800
-Wire Wire Line
-	6000 1800 6000 2000
-Text Label 6000 2000 3    50   ~ 0
+Wire Wire Line
+	5600 1800 5700 1800
+Wire Wire Line
+	6200 1800 6200 2000
+Text Label 6200 2000 3    50   ~ 0
 -12V
-Text Label 6000 1450 1    50   ~ 0
+Text Label 6200 1450 1    50   ~ 0
 +12V
-Text Notes 5350 2250 0    50   ~ 0
-adjust \nRB1/RB2 \nfor center \noffset
-$Comp
-L Device:R RB1
-U 1 1 5BB66B1F
-P 5800 1600
-F 0 "RB1" V 5700 1550 50  0000 L CNN
-F 1 "147K" V 5800 1500 50  0000 L CNN
-F 2 "Resistor_SMD:R_0805_2012Metric_Pad1.15x1.40mm_HandSolder" V 5730 1600 50  0001 C CNN
-F 3 "~" H 5800 1600 50  0001 C CNN
-	1    5800 1600
-	0    1    1    0
-$EndComp
-Wire Wire Line
-	6000 1600 6000 1450
+Wire Wire Line
+	6200 1600 6200 1450
 Wire Wire Line
 	7800 2300 7800 3100
@@
 GND
 Wire Wire Line
-	6000 1600 5950 1600
+	6200 1600 6050 1600
 Wire Wire Line
 	1950 1800 1950 1700
@@
 $EndComp
 Wire Wire Line
-	5600 1600 5650 1600
-Wire Wire Line
-	6000 1800 5950 1800
+	5600 1600 5700 1600
+Wire Wire Line
+	6200 1800 6050 1800
 Wire Wire Line
 	10100 2300 10100 2400
@@
 P 8150 2300
 F 0 "R1" V 8250 2300 50  0000 C CNN
-F 1 "1K5" V 8150 2300 50  0000 C CNN
+F 1 "390R" V 8150 2300 50  0000 C CNN
 F 2 "" V 8080 2300 50  0001 C CNN
 F 3 "~" H 8150 2300 50  0001 C CNN
@@
 	8950 2900 9200 2900
 Text Notes 8800 3650 0    50   ~ 0
-B50K
+B10K
 Text Notes 8800 2700 0    50   ~ 0
 GAIN
@@
 P 8850 4000
 F 0 "CF1" V 8601 4000 50  0000 C CNN
-F 1 "10pF" V 8690 4000 50  0000 C CNN
+F 1 "2pF" V 8690 4000 50  0000 C CNN
 F 2 "" H 8888 3850 50  0001 C CNN
 F 3 "~" H 8850 4000 50  0001 C CNN
@@
 NoConn ~ 1900 4100
 Text Notes 5050 1800 0    50   ~ 0
-B50K
+B10K
 Wire Wire Line
 	1250 1700 1250 1800
@@
 Wire Wire Line
 	1250 1800 1250 1900
+$Comp
+L Device:R_POT_TRIM OFF1
+U 1 1 5BB985CF
+P 5900 1600
+F 0 "OFF1" V 5600 1450 50  0000 C CNN
+F 1 "100K" V 5697 1600 50  0000 C CNN
+F 2 "" H 5900 1600 50  0001 C CNN
+F 3 "~" H 5900 1600 50  0001 C CNN
+	1    5900 1600
+	0    -1   -1   0
+$EndComp
+$Comp
+L Device:R_POT_TRIM OFF2
+U 1 1 5BB9865B
+P 5900 1800
+F 0 "OFF2" V 5550 1950 50  0000 C CNN
+F 1 "100K" V 5700 1800 50  0000 C CNN
+F 2 "" H 5900 1800 50  0001 C CNN
+F 3 "~" H 5900 1800 50  0001 C CNN
+	1    5900 1800
+	0    1    1    0
+$EndComp
+Wire Wire Line
+	5900 1450 5900 1400
+Wire Wire Line
+	5900 1400 5700 1400
+Wire Wire Line
+	5700 1400 5700 1600
+Connection ~ 5700 1600
+Wire Wire Line
+	5700 1600 5750 1600
+Wire Wire Line
+	5900 2000 5700 2000
+Wire Wire Line
+	5700 2000 5700 1800
+Connection ~ 5700 1800
+Wire Wire Line
+	5700 1800 5750 1800
+Wire Wire Line
+	5900 2000 5900 1950
 $EndSCHEMATC

Commit message: updates
Connections:
- net labels added: DDSOUT
Other:
- moved on the sheet: U2
Changed lines of the file:
@@
 Text Label 2150 2000 2    50   ~ 0
 -12V
-Text Label 5300 4450 0    50   ~ 0
+Text Label 5300 4800 0    50   ~ 0
 FUNCSIG
 Wire Wire Line
@@
 	1850 5950 1950 5950
 Wire Wire Line
-	5650 4450 5300 4450
+	5650 4800 5300 4800
 $Comp
 L Potentiometer_Digital:MCP42050 U2
 U 1 1 5BB5DA86
-P 6150 4750
-F 0 "U2" H 5750 5400 50  0000 C CNN
-F 1 "MCP42050" H 5750 5300 50  0000 C CNN
-F 2 "" H 6150 4850 50  0001 C CNN
-F 3 "http://ww1.microchip.com/downloads/en/DeviceDoc/11195c.pdf" H 6150 4850 50  0001 C CNN
-	1    6150 4750
+P 6150 5100
+F 0 "U2" H 5750 5750 50  0000 C CNN
+F 1 "MCP42050" H 5750 5650 50  0000 C CNN
+F 2 "" H 6150 5200 50  0001 C CNN
+F 3 "http://ww1.microchip.com/downloads/en/DeviceDoc/11195c.pdf" H 6150 5200 50  0001 C CNN
+	1    6150 5100
 	-1   0    0    -1
 $EndComp
 Wire Wire Line
-	6650 4450 6900 4450
-Text Label 6900 4450 2    50   ~ 0
+	6650 4800 6900 4800
+Text Label 6900 4800 2    50   ~ 0
 SCK
 Wire Wire Line
-	6650 4550 6900 4550
-Text Label 6900 4550 2    50   ~ 0
+	6650 4900 6900 4900
+Text Label 6900 4900 2    50   ~ 0
 MOSI
-NoConn ~ 6650 4650
-Wire Wire Line
-	6650 4750 6950 4750
-Text Label 6950 4750 2    50   ~ 0
+NoConn ~ 6650 5000
+Wire Wire Line
+	6650 5100 6950 5100
+Text Label 6950 5100 2    50   ~ 0
 POT_CS
 Wire Wire Line
@@
 POT_CS
 Wire Wire Line
-	6650 4950 7050 4950
-Wire Wire Line
-	6650 5050 7050 5050
-Wire Wire Line
-	6150 4250 6150 4000
-Text Label 6150 4000 2    50   ~ 0
+	6650 5300 7050 5300
+Wire Wire Line
+	6650 5400 7050 5400
+Wire Wire Line
+	6150 4600 6150 4350
+Text Label 6150 4350 2    50   ~ 0
 5V
 Wire Wire Line
-	6150 5250 6150 5500
-Text Label 6150 5500 2    50   ~ 0
+	6150 5600 6150 5850
+Text Label 6150 5850 2    50   ~ 0
 GND
-NoConn ~ 5650 4850
-NoConn ~ 5650 4950
-NoConn ~ 5650 5050
-Wire Wire Line
-	5650 4650 5300 4650
-Wire Wire Line
-	5300 4650 5300 4800
-Text Label 5300 4800 1    50   ~ 0
+NoConn ~ 5650 5200
+NoConn ~ 5650 5300
+NoConn ~ 5650 5400
+Wire Wire Line
+	5650 5000 5300 5000
+Wire Wire Line
+	5300 5000 5300 5150
+Text Label 5300 5150 1    50   ~ 0
 GND
 Wire Wire Line
-	7050 5050 7050 4950
-Connection ~ 7050 4950
-Wire Wire Line
-	7050 4950 7050 4800
-Text Label 7050 4800 3    50   ~ 0
+	7050 5400 7050 5300
+Connection ~ 7050 5300
+Wire Wire Line
+	7050 5300 7050 5150
+Text Label 7050 5150 3    50   ~ 0
 5V
 Wire Wire Line
@@
 Connection ~ 6400 3100
 Wire Wire Line
-	5200 3000 5200 4550
-Wire Wire Line
-	5200 4550 5650 4550
+	5200 3000 5200 4900
+Wire Wire Line
+	5200 4900 5650 4900
 Wire Wire Line
 	5200 3000 5600 3000
@@
 Wire Wire Line
 	5900 2000 5900 1950
+Text Label 5200 3000 0    50   ~ 0
+DDSOUT
 $EndSCHEMATC

Commit message: Added custom opamp symbols
Parts:
- removed U_BUFF1, U_GAIN1, U_MIX1: TL071, symbol Amplifier_Operational:TL071
- added U_BUF1: TL071, symbol Amplifier_Custom:TL071
- added U_GAIN1, U_MIX1: LM7171, symbol Amplifier_Custom:LM7171
Connections:
- wire segments 165 -> 167
- no-connect marks 25 -> 19
Other:
- note removed: "GAIN"
- note removed: "LM7171"
- note removed: "MIXER"
