File: Hardware/AD9833FunctionGenerator.sch (KiCad schematic (older format))
At the start: 33 parts, among them U1 LM7805_TO220, U2 MCP42050

Commit message: updated hardware
Parts:
- removed J_AMP1, J_OFFSET1: Conn_01x03, Connector_PinSocket_2.54mm:PinSocket_1x03_P2.54mm_Vertical, symbol Connector_Generic:Conn_01x03
- removed J_FREQ1, J_FREQ2: Conn_01x03, Connector_PinSocket_2.54mm:PinSocket_1x03_P2.54mm_Vertical, symbol AD9833FunctionGenerator-rescue:Conn_01x03
- removed R1: 390R, symbol Device:R
- added C_GAIN2: 470pF, symbol Device:C
- added C_MIXF1, C_MIXIN1: ?, symbol Device:C
- added RV_FREQ1, RV_FREQ2, RV_OFF1: B10K, symbol Device:R_POT_Dual_Separate
- added RV_GAIN1: R_POT_Dual_Separate, symbol Device:R_POT_Dual_Separate
- added RV_LOWG1: 100R, symbol Device:R_POT_TRIM
- added RV_TOPG1: 10K, symbol Device:R_POT_TRIM
- added R_LOWG1: 120R, symbol Device:R
- added R_TOPG1: 330R, symbol Device:R
- C_GAINF1: renamed from CF1; value 2pF -> ?
- R_ISO1: value 330R -> 600R 1%
- renumbered RF1 to R_MIXF1
Connections:
- wire segments 167 -> 194
Other:
- note removed: "10K Pot"
- note removed: "B10K"
- moved on the sheet: U2

Commit message: Created board layout RevB. Right-angled to front panel, with front facing aux board(OLED/Buttons)
Parts:
- removed J_OLED1: Conn_01x04, Connector_PinSocket_2.54mm:PinSocket_1x04_P2.54mm_Vertical, symbol AD9833FunctionGenerator-rescue:Conn_01x04
- removed J_TX1, J_VIN1: Conn_01x15, Connector_PinSocket_2.54mm:PinSocket_1x15_P2.54mm_Vertical, symbol AD9833FunctionGenerator-rescue:Conn_01x15
- removed J_VEL1: Conn_01x03, Connector_PinSocket_2.54mm:PinSocket_1x03_P2.54mm_Vertical, symbol AD9833FunctionGenerator-rescue:Conn_01x03
- removed R_FUNC1, R_MODE1, R_RANGE1: 1K, Resistor_SMD:R_0805_2012Metric_Pad1.15x1.40mm_HandSolder, symbol Device:R
- removed SW_FUNC1, SW_MODE1, SW_RANGE1: SW_SPST, Button_Switch_THT:SW_PUSH_6mm, symbol Switch:SW_SPST
- added A1: Arduino_Nano_v3.x, Module:Arduino_Nano, symbol MCU_Module:Arduino_Nano_v3.x
- added C_BUFBP1, C_BUFBP2: 100nF, Capacitor_SMD:C_0805_2012Metric_Pad1.15x1.40mm_HandSolder, symbol Device:C
- added C_GAINBP1, C_GAINBP3, C_MIXBP1, C_MIXBP3: 10nF, Capacitor_SMD:C_0805_2012Metric_Pad1.15x1.40mm_HandSolder, symbol Device:C
- added C_GAINBP2, C_GAINBP4, C_MIXBP2: 2.2uF TANT., Capacitor_SMD:C_0805_2012Metric_Pad1.15x1.40mm_HandSolder, symbol Device:CP
- added C_MIXBP4: 2.2pF TANT., Capacitor_SMD:C_0805_2012Metric_Pad1.15x1.40mm_HandSolder, symbol Device:CP
- added J_MAIN2AUX1: Conn_02x05_Odd_Even, Connector_PinHeader_2.54mm:PinHeader_2x05_P2.54mm_Vertical, symbol Connector_Generic:Conn_02x05_Odd_Even
- added RV_TIME1: B10K, PTH901:PTH901, symbol Device:R_POT_Dual_Separate
- C_GAIN2, C_GAINF1, C_MIXF1, C_MIXIN1: footprint (none) -> Capacitor_SMD:C_0805_2012Metric_Pad1.15x1.40mm_HandSolder
- RV_AMP1: renamed from RV_OFF1; footprint (none) -> PTH901:PTH901; MouserPartNo (none) -> 652-PTH901-030S-103B
- RV_AMP1: renamed from RV_GAIN1; value R_POT_Dual_Separate -> B10K; footprint (none) -> PTH901:PTH901; MouserPartNo (none) -> 652-PTH901-030S-103B
- RV_FREQ1: renamed from RV_FREQ2; footprint (none) -> PTH901:PTH901; MouserPartNo (none) -> 652-PTH901-030S-103B
- RV_FREQ1: footprint (none) -> PTH901:PTH901; MouserPartNo (none) -> 652-PTH901-030S-103B
- RV_LOWG1: footprint (none) -> Potentiometer_THT:Potentiometer_Bourns_3296Y_Vertical; MouserPartNo (none) -> 652-3296Y-1-101LF
- RV_LOWOFF1: renamed from OFF2; footprint (none) -> Potentiometer_THT:Potentiometer_Bourns_3296Y_Vertical; MouserPartNo (none) -> 652-3296Y-1-104LF
- RV_TOPG1: footprint (none) -> Potentiometer_THT:Potentiometer_Bourns_3296Y_Vertical; MouserPartNo (none) -> 652-3296Y-1-103LF
- RV_UPOFF1: renamed from OFF1; footprint (none) -> Potentiometer_THT:Potentiometer_Bourns_3296Y_Vertical; MouserPartNo (none) -> 652-3296Y-1-104LF
- R_ISO1, R_LOWG1, R_MIXF1, R_TOPG1: footprint (none) -> Resistor_SMD:R_0805_2012Metric_Pad1.15x1.40mm_HandSolder
- U1: MouserPartNo (none) -> 926-LM7805CT/NOPB
- U_BUF1: footprint (none) -> Package_SO:SOIC-8_3.9x4.9mm_P1.27mm; MouserPartNo (none) -> 595-TL071ACDR
- U_GAIN1, U_MIX1: footprint (none) -> Package_SO:SOIC-8_3.9x4.9mm_P1.27mm; MouserPartNo (none) -> 926-LM7171BIMX/NOPB
- U_POT1: renamed from U2; footprint (none) -> Package_SO:SOIC-14_3.9x8.7mm_P1.27mm; MouserPartNo (none) -> 579-MCP42050-I/SL
Connections:
- net labels added: AREF, MODEBTN, RANGEBTN, WAVEBTN
- net labels removed: FUNCMODE1, RANGEMODE1, SWEEPMODE1
- wire segments 194 -> 218
- no-connect marks 19 -> 24
Other:
- note added: "Auxiliary Board"
- note added: "Output Section"
- note removed: "Arduino Nano sockets"
- note removed: "BUFFER"
- note removed: "OUTPUT"
- note removed: "TX\nRX\nRST\nGND\nD2\nD3\nD4\nD5\nD6\nD7\nD8\nD9\nD10\nD11\nD12"
- note removed: "VIN\nGND\nRST\n5V\nA7\nA6\nA5\nA4\nA3\nA2\nA1\nA0\nAREF\n3V3\nD13"
- moved on the sheet: U_POT1

Commit message: Tidied up schematic. Added sub-sheets
Parts:
- removed C_BUFBP1, C_BUFBP2: 100nF, Capacitor_SMD:C_0805_2012Metric_Pad1.15x1.40mm_HandSolder, symbol Device:C
- removed C_GAIN2: 470pF, Capacitor_SMD:C_0805_2012Metric_Pad1.15x1.40mm_HandSolder, symbol Device:C
- removed C_GAINBP1, C_GAINBP3, C_MIXBP1, C_MIXBP3: 10nF, Capacitor_SMD:C_0805_2012Metric_Pad1.15x1.40mm_HandSolder, symbol Device:C
- removed C_GAINBP2, C_GAINBP4, C_MIXBP2: 2.2uF TANT., Capacitor_SMD:C_0805_2012Metric_Pad1.15x1.40mm_HandSolder, symbol Device:CP
- removed C_GAINF1, C_MIXF1, C_MIXIN1: ?, Capacitor_SMD:C_0805_2012Metric_Pad1.15x1.40mm_HandSolder, symbol Device:C
- removed C_MIXBP4: 2.2pF TANT., Capacitor_SMD:C_0805_2012Metric_Pad1.15x1.40mm_HandSolder, symbol Device:CP
- removed J_MAIN2AUX1: Conn_02x05_Odd_Even, Connector_PinHeader_2.54mm:PinHeader_2x05_P2.54mm_Vertical, symbol Connector_Generic:Conn_02x05_Odd_Even
- removed RV_AMP1: B10K, PTH901:PTH901, symbol Device:R_POT_Dual_Separate
- removed RV_LOWG1: 100R, Potentiometer_THT:Potentiometer_Bourns_3296Y_Vertical, symbol Device:R_POT_TRIM
- removed RV_LOWOFF1, RV_UPOFF1: 100K, Potentiometer_THT:Potentiometer_Bourns_3296Y_Vertical, symbol Device:R_POT_TRIM
- removed RV_TOPG1: 10K, Potentiometer_THT:Potentiometer_Bourns_3296Y_Vertical, symbol Device:R_POT_TRIM
- removed R_ISO1: 600R 1%, Resistor_SMD:R_0805_2012Metric_Pad1.15x1.40mm_HandSolder, symbol Device:R
- removed R_LOWG1: 120R, Resistor_SMD:R_0805_2012Metric_Pad1.15x1.40mm_HandSolder, symbol Device:R
- removed R_MIX1, R_MIX2, R_MIXF1: 10K, Resistor_SMD:R_0805_2012Metric_Pad1.15x1.40mm_HandSolder, symbol Device:R
- removed R_TOPG1: 330R, Resistor_SMD:R_0805_2012Metric_Pad1.15x1.40mm_HandSolder, symbol Device:R
- removed U_BUF1: TL071, Package_SO:SOIC-8_3.9x4.9mm_P1.27mm, symbol Amplifier_Custom:TL071
- removed U_GAIN1, U_MIX1: LM7171, Package_SO:SOIC-8_3.9x4.9mm_P1.27mm, symbol Amplifier_Custom:LM7171
Connections:
- net labels added: DDS_REDUX, DDS_SIG
- net labels removed: DDSOUT, FUNCSIG
- wire segments 218 -> 104
- no-connect marks 24 -> 21
Other:
- note added: "DDS Signal Generation"
- note added: "Output Amplifier Section"
- note added: "Peripheral Controls section"
- note added: "Power Supply Section"
- note removed: "Auxiliary Board"
- note removed: "Output Section"
- note removed: "Power supply"
- moved on the sheet: U_POT1

Commit message: updates
Other:
- note added: "Micocontroller"
- note added: "Signal Compensation"
- moved on the sheet: U_POT1

Commit message: updated HW
- Added separate analog and digital ground to prevent output signal ripple/jitter
Parts:
- added C_POTBP1: 100nF, Capacitor_SMD:C_0805_2012Metric_Pad1.15x1.40mm_HandSolder, symbol Device:C
Connections:
- net labels added: AGND
- wire segments 104 -> 108
Other:
- moved on the sheet: U_POT1
Changed lines of the file:
@@
 	2750 6700 3350 6700
 Text Label 2750 6950 2    50   ~ 0
-GND
+AGND
 Text Label 2850 6400 0    50   ~ 0
 FREQ1
@@
 MODEBTN
 Text Label 4850 5500 2    50   ~ 0
-GND
+AGND
 Text Label 4850 4200 2    50   ~ 0
 5V
@@
 Text Label 2600 1850 2    50   ~ 0
 -12V
-Text Label 5650 1650 0    50   ~ 0
+Text Label 5900 1850 0    50   ~ 0
 DDS_SIG
 $Comp
@@
 	10500 2150 10350 2150
 Text Label 10350 2800 2    50   ~ 0
-GND
+AGND
 Wire Wire Line
 	2300 1650 2300 1550
@@
 +12V
 Text Label 900  1650 0    50   ~ 0
-GND
+AGND
 Text Label 900  1850 0    50   ~ 0
 -12V
@@
 RANGEBTN
 Wire Wire Line
-	6050 1650 5650 1650
+	6300 1850 5900 1850
 $Comp
 L Potentiometer_Digital:MCP42050 U_POT1
 U 1 1 5BB5DA86
-P 6550 1950
-F 0 "U_POT1" H 6150 2600 50  0000 C CNN
-F 1 "MCP42050" H 6150 2500 50  0000 C CNN
-F 2 "Package_SO:SOIC-14_3.9x8.7mm_P1.27mm" H 6550 2050 50  0001 C CNN
-F 3 "http://ww1.microchip.com/downloads/en/DeviceDoc/11195c.pdf" H 6550 2050 50  0001 C CNN
-F 4 "579-MCP42050-I/SL" H 700 -3150 50  0001 C CNN "MouserPartNo"
-	1    6550 1950
+P 6800 2150
+F 0 "U_POT1" H 6400 2800 50  0000 C CNN
+F 1 "MCP42050" H 6400 2700 50  0000 C CNN
+F 2 "Package_SO:SOIC-14_3.9x8.7mm_P1.27mm" H 6800 2250 50  0001 C CNN
+F 3 "http://ww1.microchip.com/downloads/en/DeviceDoc/11195c.pdf" H 6800 2250 50  0001 C CNN
+F 4 "579-MCP42050-I/SL" H 950 -2950 50  0001 C CNN "MouserPartNo"
+	1    6800 2150
 	-1   0    0    -1
 $EndComp
 Wire Wire Line
-	7050 1650 7250 1650
-Text Label 7250 1650 2    50   ~ 0
+	7300 1850 7500 1850
+Text Label 7500 1850 2    50   ~ 0
 SCK
 Wire Wire Line
-	7050 1750 7250 1750
-Text Label 7250 1750 2    50   ~ 0
+	7300 1950 7500 1950
+Text Label 7500 1950 2    50   ~ 0
 MOSI
-NoConn ~ 7050 1850
-Wire Wire Line
-	7050 1950 7300 1950
-Text Label 7300 1950 2    50   ~ 0
+NoConn ~ 7300 2050
+Wire Wire Line
+	7300 2150 7550 2150
+Text Label 7550 2150 2    50   ~ 0
 POT_CS
 Wire Wire Line
@@
 POT_CS
 Wire Wire Line
-	7050 2150 7150 2150
-Wire Wire Line
-	7050 2250 7150 2250
-Wire Wire Line
-	6550 1450 6550 1400
-Text Label 6550 1400 2    50   ~ 0
+	7300 2350 7400 2350
+Wire Wire Line
+	7300 2450 7400 2450
+Wire Wire Line
+	6800 1650 6800 1450
+Text Label 6800 1300 2    50   ~ 0
 5V
 Wire Wire Line
-	6550 2450 6550 2600
-Text Label 6550 2600 2    50   ~ 0
+	6800 2650 6800 2800
+Text Label 6800 2800 2    50   ~ 0
 GND
-NoConn ~ 6050 2050
-NoConn ~ 6050 2150
-NoConn ~ 6050 2250
-Text Label 5900 2600 0    50   ~ 0
+NoConn ~ 6300 2250
+NoConn ~ 6300 2350
+NoConn ~ 6300 2450
+Text Label 6150 2800 0    50   ~ 0
 GND
 Wire Wire Line
-	7150 2250 7150 2150
-Connection ~ 7150 2150
-Wire Wire Line
-	7150 2150 7300 2150
-Text Label 7300 2150 2    50   ~ 0
+	7400 2450 7400 2350
+Connection ~ 7400 2350
+Wire Wire Line
+	7400 2350 7550 2350
+Text Label 7550 2350 2    50   ~ 0
 5V
 Wire Wire Line
-	5650 1750 6050 1750
+	5900 1950 6300 1950
 Wire Wire Line
 	10350 2150 10350 2800
@@
 NoConn ~ 9900 4350
 NoConn ~ 9600 3950
-Text Label 5650 1750 0    50   ~ 0
+Text Label 5900 1950 0    50   ~ 0
 DDS_REDUX
 Wire Wire Line
@@
 F3 "+12V" I L 9100 1550 50
 F4 "-12V" I L 9100 1650 50
-F5 "GND" I L 9100 2450 50
-F6 "SIGOUT" I R 10150 2050 50
+F5 "SIGOUT" I R 10150 2050 50
+F6 "AGND" I L 9100 2450 50
 $EndSheet
 Text Label 1750 3100 2    50   ~ 0
@@
 	8850 2450 8850 2800
 Text Label 8850 2800 2    50   ~ 0
-GND
+AGND
 Wire Wire Line
 	9100 1550 8950 1550
@@
 5V
 Wire Wire Line
-	5900 2600 5900 1850
-Wire Wire Line
-	5900 1850 6050 1850
+	6150 2800 6150 2050
+Wire Wire Line
+	6150 2050 6300 2050
 Wire Wire Line
 	8600 2050 9100 2050
@@
 Text Notes 8200 3550 0    50   ~ 0
 Micocontroller
+$Comp
+L Device:C C_POTBP1
+U 1 1 5BC0F1E8
+P 5900 1450
+F 0 "C_POTBP1" V 5651 1450 50  0000 C CNN
+F 1 "100nF" V 5740 1450 50  0000 C CNN
+F 2 "Capacitor_SMD:C_0805_2012Metric_Pad1.15x1.40mm_HandSolder" H 5938 1300 50  0001 C CNN
+F 3 "~" H 5900 1450 50  0001 C CNN
+	1    5900 1450
+	0    1    1    0
+$EndComp
+Wire Wire Line
+	6050 1450 6800 1450
+Connection ~ 6800 1450
+Wire Wire Line
+	6800 1450 6800 1300
+Wire Wire Line
+	5750 1450 5600 1450
+Wire Wire Line
+	5600 1450 5600 2800
+Text Label 5600 2800 0    50   ~ 0
+GND
 $EndSCHEMATC

Commit message: updates
Parts:
- added ROFF1, ROFF2: 1K, symbol Device:R
Connections:
- net labels added: OFFSETADJUST
- wire segments 108 -> 116
- no-connect marks 21 -> 18
Other:
- moved on the sheet: U_POT1
Changed lines of the file:
@@
 L AD9833FunctionGenerator-rescue:Conn_01x07 J_AD9833
 U 1 1 5B8B29C3
-P 4350 1950
-F 0 "J_AD9833" H 4350 2500 50  0000 C CNN
-F 1 "Conn_01x07" H 4350 2400 50  0000 C CNN
-F 2 "Connector_PinSocket_2.54mm:PinSocket_1x07_P2.54mm_Vertical" H 4350 1950 50  0001 C CNN
-F 3 "" H 4350 1950 50  0001 C CNN
-	1    4350 1950
+P 3900 1950
+F 0 "J_AD9833" H 3900 2500 50  0000 C CNN
+F 1 "Conn_01x07" H 3900 2400 50  0000 C CNN
+F 2 "Connector_PinSocket_2.54mm:PinSocket_1x07_P2.54mm_Vertical" H 3900 1950 50  0001 C CNN
+F 3 "" H 3900 1950 50  0001 C CNN
+	1    3900 1950
 	1    0    0    -1
 $EndComp
@@
 SCK
 Wire Wire Line
-	4150 1750 3700 1750
-Wire Wire Line
-	4150 1850 3700 1850
-Wire Wire Line
-	4150 1950 3700 1950
-Wire Wire Line
-	4150 2050 3700 2050
-Wire Wire Line
-	4150 2150 3700 2150
-Wire Wire Line
-	4150 2250 3700 2250
-Text Notes 4450 2300 0    63   ~ 0
+	3700 1750 3250 1750
+Wire Wire Line
+	3700 1850 3250 1850
+Wire Wire Line
+	3700 1950 3250 1950
+Wire Wire Line
+	3700 2050 3250 2050
+Wire Wire Line
+	3700 2150 3250 2150
+Wire Wire Line
+	3700 2250 3250 2250
+Text Notes 4000 2300 0    63   ~ 0
 REF\nVCC\nGND\nDAT\nCLK\nFNC\nOUT
-NoConn ~ 4150 1650
-Text Label 3700 1750 0    50   ~ 0
-5V
-Text Label 3700 1850 0    50   ~ 0
+NoConn ~ 3700 1650
+Text Label 3250 1750 0    50   ~ 0
+5V
+Text Label 3250 1850 0    50   ~ 0
 GND
-Text Label 3700 1950 0    50   ~ 0
+Text Label 3250 1950 0    50   ~ 0
 MOSI
-Text Label 3700 2050 0    50   ~ 0
+Text Label 3250 2050 0    50   ~ 0
 SCK
-Text Label 3700 2150 0    50   ~ 0
+Text Label 3250 2150 0    50   ~ 0
 DDS_CS
-Text Label 3700 2250 0    50   ~ 0
+Text Label 3250 2250 0    50   ~ 0
 DDS_SIG
 Wire Wire Line
@@
 Text Label 2600 1850 2    50   ~ 0
 -12V
-Text Label 5900 1850 0    50   ~ 0
+Text Label 6100 1850 0    50   ~ 0
 DDS_SIG
 $Comp
@@
 RANGEBTN
 Wire Wire Line
-	6300 1850 5900 1850
+	6500 1850 6100 1850
 $Comp
 L Potentiometer_Digital:MCP42050 U_POT1
 U 1 1 5BB5DA86
-P 6800 2150
-F 0 "U_POT1" H 6400 2800 50  0000 C CNN
-F 1 "MCP42050" H 6400 2700 50  0000 C CNN
-F 2 "Package_SO:SOIC-14_3.9x8.7mm_P1.27mm" H 6800 2250 50  0001 C CNN
-F 3 "http://ww1.microchip.com/downloads/en/DeviceDoc/11195c.pdf" H 6800 2250 50  0001 C CNN
-F 4 "579-MCP42050-I/SL" H 950 -2950 50  0001 C CNN "MouserPartNo"
-	1    6800 2150
+P 7000 2150
+F 0 "U_POT1" H 6600 2800 50  0000 C CNN
+F 1 "MCP42050" H 6600 2700 50  0000 C CNN
+F 2 "Package_SO:SOIC-14_3.9x8.7mm_P1.27mm" H 7000 2250 50  0001 C CNN
+F 3 "http://ww1.microchip.com/downloads/en/DeviceDoc/11195c.pdf" H 7000 2250 50  0001 C CNN
+F 4 "579-MCP42050-I/SL" H 1150 -2950 50  0001 C CNN "MouserPartNo"
+	1    7000 2150
 	-1   0    0    -1
 $EndComp
 Wire Wire Line
-	7300 1850 7500 1850
-Text Label 7500 1850 2    50   ~ 0
+	7500 1850 7700 1850
+Text Label 7700 1850 2    50   ~ 0
 SCK
 Wire Wire Line
-	7300 1950 7500 1950
-Text Label 7500 1950 2    50   ~ 0
+	7500 1950 7700 1950
+Text Label 7700 1950 2    50   ~ 0
 MOSI
-NoConn ~ 7300 2050
-Wire Wire Line
-	7300 2150 7550 2150
-Text Label 7550 2150 2    50   ~ 0
+NoConn ~ 7500 2050
+Wire Wire Line
+	7500 2150 7750 2150
+Text Label 7750 2150 2    50   ~ 0
 POT_CS
 Wire Wire Line
@@
 POT_CS
 Wire Wire Line
-	7300 2350 7400 2350
-Wire Wire Line
-	7300 2450 7400 2450
-Wire Wire Line
-	6800 1650 6800 1450
-Text Label 6800 1300 2    50   ~ 0
-5V
-Wire Wire Line
-	6800 2650 6800 2800
-Text Label 6800 2800 2    50   ~ 0
+	7500 2350 7600 2350
+Wire Wire Line
+	7500 2450 7600 2450
+Wire Wire Line
+	7000 1650 7000 1450
+Text Label 7000 1300 2    50   ~ 0
+5V
+Wire Wire Line
+	7000 2650 7000 2800
+Text Label 7000 2800 2    50   ~ 0
 GND
-NoConn ~ 6300 2250
-NoConn ~ 6300 2350
-NoConn ~ 6300 2450
-Text Label 6150 2800 0    50   ~ 0
-GND
-Wire Wire Line
-	7400 2450 7400 2350
-Connection ~ 7400 2350
-Wire Wire Line
-	7400 2350 7550 2350
-Text Label 7550 2350 2    50   ~ 0
-5V
-Wire Wire Line
-	5900 1950 6300 1950
+Wire Wire Line
+	7600 2450 7600 2350
+Connection ~ 7600 2350
+Wire Wire Line
+	7600 2350 7750 2350
+Text Label 7750 2350 2    50   ~ 0
+5V
+Wire Wire Line
+	6100 1950 6500 1950
 Wire Wire Line
 	10350 2150 10350 2800
@@
 NoConn ~ 9900 4350
 NoConn ~ 9600 3950
-Text Label 5900 1950 0    50   ~ 0
+Text Label 6100 1950 0    50   ~ 0
 DDS_REDUX
 Wire Wire Line
@@
 F5 "SIGOUT" I R 10150 2050 50
 F6 "AGND" I L 9100 2450 50
+F7 "OFFSETADJUST" I L 9100 1850 50
 $EndSheet
 Text Label 1750 3100 2    50   ~ 0
@@
 	2300 6400 2650 6400
 Wire Notes Line
-	3600 1000 3600 2800
-Wire Notes Line
-	4750 2800 4750 1000
-Wire Notes Line
-	4750 1000 3600 1000
+	3150 1000 3150 2800
+Wire Notes Line
+	4300 2800 4300 1000
+Wire Notes Line
+	4300 1000 3150 1000
 Wire Notes Line
 	10900 3100 10900 1000
@@
 Wire Notes Line
 	2900 1000 700  1000
-Text Notes 3600 950  0    50   ~ 0
+Text Notes 3150 950  0    50   ~ 0
 DDS Signal Generation
 Text Notes 8400 950  0    50   ~ 0
@@
 5V
 Wire Wire Line
-	6150 2800 6150 2050
-Wire Wire Line
-	6150 2050 6300 2050
-Wire Wire Line
-	8600 2050 9100 2050
-Text Label 8600 2050 0    50   ~ 0
+	5000 2050 6500 2050
+Wire Wire Line
+	8500 2050 9100 2050
+Text Label 8500 2050 0    50   ~ 0
 DDS_REDUX
 Wire Notes Line
-	3600 2800 4750 2800
-Wire Notes Line
-	5400 1000 7700 1000
-Wire Notes Line
-	7700 1000 7700 3100
-Wire Notes Line
-	7700 3100 5400 3100
-Wire Notes Line
-	5400 3100 5400 1000
-Text Notes 5400 950  0    50   ~ 0
+	3150 2800 4300 2800
+Wire Notes Line
+	4800 1000 7900 1000
+Wire Notes Line
+	7900 1000 7900 3100
+Wire Notes Line
+	7900 3100 4800 3100
+Wire Notes Line
+	4800 3100 4800 1000
+Text Notes 5600 950  0    50   ~ 0
 Signal Compensation
 Text Notes 8200 3550 0    50   ~ 0
@@
 L Device:C C_POTBP1
 U 1 1 5BC0F1E8
-P 5900 1450
-F 0 "C_POTBP1" V 5651 1450 50  0000 C CNN
-F 1 "100nF" V 5740 1450 50  0000 C CNN
-F 2 "Capacitor_SMD:C_0805_2012Metric_Pad1.15x1.40mm_HandSolder" H 5938 1300 50  0001 C CNN
-F 3 "~" H 5900 1450 50  0001 C CNN
-	1    5900 1450
+P 6100 1450
+F 0 "C_POTBP1" V 5851 1450 50  0000 C CNN
+F 1 "100nF" V 5940 1450 50  0000 C CNN
+F 2 "Capacitor_SMD:C_0805_2012Metric_Pad1.15x1.40mm_HandSolder" H 6138 1300 50  0001 C CNN
+F 3 "~" H 6100 1450 50  0001 C CNN
+	1    6100 1450
 	0    1    1    0
 $EndComp
 Wire Wire Line
-	6050 1450 6800 1450
-Connection ~ 6800 1450
-Wire Wire Line
-	6800 1450 6800 1300
-Wire Wire Line
-	5750 1450 5600 1450
-Wire Wire Line
-	5600 1450 5600 2800
-Text Label 5600 2800 0    50   ~ 0
+	6250 1450 7000 1450
+Connection ~ 7000 1450
+Wire Wire Line
+	7000 1450 7000 1300
+Wire Wire Line
+	5950 1450 5000 1450
+Wire Wire Line
+	5000 1450 5000 2050
+Text Label 5000 2800 0    50   ~ 0
 GND
+Connection ~ 5000 2050
+Wire Wire Line
+	5000 2050 5000 2800
+Wire Wire Line
+	6500 2450 6300 2450
+Wire Wire Line
+	6500 2350 5200 2350
+$Comp
+L Device:R ROFF1
+U 1 1 5BC66CD0
+P 6150 2250
+F 0 "ROFF1" V 6050 2250 50  0000 C CNN
+F 1 "1K" V 6150 2250 50  0000 C CNN
+F 2 "" V 6080 2250 50  0001 C CNN
+F 3 "~" H 6150 2250 50  0001 C CNN
+	1    6150 2250
+	0    1    1    0
+$EndComp
+Wire Wire Line
+	6300 2250 6500 2250
+$Comp
+L Device:R ROFF2
+U 1 1 5BC6A9D4
+P 6150 2450
+F 0 "ROFF2" V 6250 2450 50  0000 C CNN
+F 1 "1K" V 6150 2450 50  0000 C CNN
+F 2 "" V 6080 2450 50  0001 C CNN
+F 3 "~" H 6150 2450 50  0001 C CNN
+	1    6150 2450
+	0    1    1    0
+$EndComp
+Wire Wire Line
+	6000 2250 5750 2250
+Wire Wire Line
+	5750 2250 5750 2075
+Text Label 5750 2075 3    50   ~ 0
++12V
+Wire Wire Line
+	6000 2450 5750 2450
+Wire Wire Line
+	5750 2450 5750 2625
+Text Label 5750 2625 1    50   ~ 0
+-12V
+Text Label 5200 2350 0    50   ~ 0
+OFFSETADJUST
+Wire Wire Line
+	9100 1850 8500 1850
+Text Label 8500 1850 0    50   ~ 0
+OFFSETADJUST
 $EndSCHEMATC

Commit message: board rev b
Parts:
- ROFF1, ROFF2: footprint (none) -> Resistor_SMD:R_0805_2012Metric_Pad1.15x1.40mm_HandSolder
Changed lines of the file:
@@
 Text Label 2600 1850 2    50   ~ 0
 -12V
-Text Label 6100 1850 0    50   ~ 0
+Text Label 5200 1850 0    50   ~ 0
 DDS_SIG
 $Comp
@@
 RANGEBTN
 Wire Wire Line
-	6500 1850 6100 1850
+	6500 1850 5200 1850
 $Comp
 L Potentiometer_Digital:MCP42050 U_POT1
@@
 5V
 Wire Wire Line
-	6100 1950 6500 1950
+	5200 1950 6500 1950
 Wire Wire Line
 	10350 2150 10350 2800
@@
 NoConn ~ 9900 4350
 NoConn ~ 9600 3950
-Text Label 6100 1950 0    50   ~ 0
+Text Label 5200 1950 0    50   ~ 0
 DDS_REDUX
 Wire Wire Line
@@
 5V
 Wire Wire Line
-	5000 2050 6500 2050
-Wire Wire Line
 	8500 2050 9100 2050
 Text Label 8500 2050 0    50   ~ 0
@@
 Wire Wire Line
 	5950 1450 5000 1450
-Wire Wire Line
-	5000 1450 5000 2050
 Text Label 5000 2800 0    50   ~ 0
 GND
-Connection ~ 5000 2050
-Wire Wire Line
-	5000 2050 5000 2800
 Wire Wire Line
 	6500 2450 6300 2450
@@
 F 0 "ROFF1" V 6050 2250 50  0000 C CNN
 F 1 "1K" V 6150 2250 50  0000 C CNN
-F 2 "" V 6080 2250 50  0001 C CNN
+F 2 "Resistor_SMD:R_0805_2012Metric_Pad1.15x1.40mm_HandSolder" V 6080 2250 50  0001 C CNN
 F 3 "~" H 6150 2250 50  0001 C CNN
 	1    6150 2250
@@
 F 0 "ROFF2" V 6250 2450 50  0000 C CNN
 F 1 "1K" V 6150 2450 50  0000 C CNN
-F 2 "" V 6080 2450 50  0001 C CNN
+F 2 "Resistor_SMD:R_0805_2012Metric_Pad1.15x1.40mm_HandSolder" V 6080 2450 50  0001 C CNN
 F 3 "~" H 6150 2450 50  0001 C CNN
 	1    6150 2450
@@
 	6000 2250 5750 2250
 Wire Wire Line
-	5750 2250 5750 2075
-Text Label 5750 2075 3    50   ~ 0
-+12V
+	5750 2250 5750 2150
+Text Label 5750 2150 3    50   ~ 0
+5V
 Wire Wire Line
 	6000 2450 5750 2450
@@
 	5750 2450 5750 2625
 Text Label 5750 2625 1    50   ~ 0
--12V
+AGND
 Text Label 5200 2350 0    50   ~ 0
 OFFSETADJUST
@@
 Text Label 8500 1850 0    50   ~ 0
 OFFSETADJUST
+Wire Wire Line
+	5000 1450 5000 2800
+Text Label 5900 2200 1    50   ~ 0
+AGND
+Wire Wire Line
+	5900 2050 5900 2200
+Wire Wire Line
+	5900 2050 6500 2050
 $EndSCHEMATC

Commit message: updated board layout
Parts:
- removed RV_TIME1: B10K, PTH901:PTH901, symbol Device:R_POT_Dual_Separate
- added RV_SPEED1: R_POT, PTD901:PTD90, symbol Device:R_POT
Connections:
- wire segments 116 -> 113
- no-connect marks 18 -> 15
Changed lines of the file:
@@
 Wire Wire Line
 	4850 5200 4850 5500
-$Comp
-L Device:R_POT_Dual_Separate RV_TIME1
-U 1 1 5C779514
-P 4850 4600
-F 0 "RV_TIME1" H 4750 4550 50  0000 R CNN
-F 1 "B10K" H 4550 4650 50  0000 R CNN
-F 2 "PTH901:PTH901" H 4850 4600 50  0001 C CNN
-F 3 "~" H 4850 4600 50  0001 C CNN
-	1    4850 4600
-	1    0    0    1
-$EndComp
-$Comp
-L Device:R_POT_Dual_Separate RV_TIME1
-U 2 1 5C79DB8E
-P 4850 6400
-F 0 "RV_TIME1" H 4750 6450 50  0000 R CNN
-F 1 "B10K" H 4550 6350 50  0000 R CNN
-F 2 "PTH901:PTH901" H 4850 6400 50  0001 C CNN
-F 3 "~" H 4850 6400 50  0001 C CNN
-	2    4850 6400
-	1    0    0    -1
-$EndComp
 $Sheet
 S 2050 3900 1400 1600
@@
 Wire Wire Line
 	4850 4200 4850 4450
-Wire Wire Line
-	4850 6250 4850 6100
-Wire Wire Line
-	5000 6400 5150 6400
-Wire Wire Line
-	4850 6550 4850 6700
-NoConn ~ 4850 6100
-NoConn ~ 4850 6700
-NoConn ~ 5150 6400
 Wire Notes Line
 	1450 7250 5550 7250
@@
 Wire Wire Line
 	5900 2050 6500 2050
+$Comp
+L Device:R_POT RV_SPEED1
+U 1 1 5BC3EBD3
+P 4850 4600
+F 0 "RV_SPEED1" H 4780 4646 50  0000 R CNN
+F 1 "R_POT" H 4780 4555 50  0000 R CNN
+F 2 "PTD901:PTD90" H 4850 4600 50  0001 C CNN
+F 3 "~" H 4850 4600 50  0001 C CNN
+	1    4850 4600
+	1    0    0    -1
+$EndComp
 $EndSCHEMATC
