File: Hardware/OutputSection.sch (KiCad schematic (older format))
At the start: 28 parts

Commit message: updates
Parts:
- added TP_OFF1: TestPoint, symbol Connector:TestPoint
Connections:
- wire segments 124 -> 125
Changed lines of the file:
@@
 Wire Wire Line
 	5850 2900 6100 2900
+$Comp
+L Connector:TestPoint TP_OFF1
+U 1 1 5BCAA241
+P 2150 2550
+F 0 "TP_OFF1" H 2207 2669 50  0000 L CNN
+F 1 "TestPoint" H 2207 2580 50  0000 L CNN
+F 2 "" H 2350 2550 50  0001 C CNN
+F 3 "~" H 2350 2550 50  0001 C CNN
+	1    2150 2550
+	1    0    0    -1
+$EndComp
+Wire Wire Line
+	2150 2550 2150 2700
+Connection ~ 2150 2700
 $EndSCHEMATC

Commit message: updated HW
- Added separate analog and digital ground to prevent output signal ripple/jitter
Parts:
- added R_HIOFF1, R_LOFF1: 220R, Resistor_SMD:R_0805_2012Metric_Pad1.15x1.40mm_HandSolder, symbol Device:R
- TP_OFF1: footprint (none) -> TestPoint:TestPoint_Pad_D2.0mm
Connections:
- net labels added: AGND
- net labels removed: GND
- wire segments 125 -> 127
Changed lines of the file:
@@
 L Device:R_POT_TRIM RV_LOWG1
 U 1 1 5BBE4810
-P 8550 1900
-F 0 "RV_LOWG1" H 9150 1900 50  0000 R CNN
-F 1 "100R" V 8550 2000 50  0000 R CNN
-F 2 "Potentiometer_THT:Potentiometer_Bourns_3296Y_Vertical" H 8550 1900 50  0001 C CNN
-F 3 "~" H 8550 1900 50  0001 C CNN
-F 4 "652-3296Y-1-101LF" H -550 -1200 50  0001 C CNN "MouserPartNo"
-	1    8550 1900
-	1    0    0    1
+P 9750 1900
+F 0 "RV_LOWG1" H 10350 1900 50  0000 R CNN
+F 1 "100R" V 9750 2000 50  0000 R CNN
+F 2 "Potentiometer_THT:Potentiometer_Bourns_3296Y_Vertical" H 9750 1900 50  0001 C CNN
+F 3 "~" H 9750 1900 50  0001 C CNN
+F 4 "652-3296Y-1-101LF" H 650 -1200 50  0001 C CNN "MouserPartNo"
+	1    9750 1900
+	-1   0    0    1
 $EndComp
 $Comp
 L Device:R R_LOWG1
 U 1 1 5BBE4817
-P 8550 1550
-F 0 "R_LOWG1" H 8620 1595 50  0000 L CNN
-F 1 "120R" V 8550 1450 50  0000 L CNN
-F 2 "Resistor_SMD:R_0805_2012Metric_Pad1.15x1.40mm_HandSolder" V 8480 1550 50  0001 C CNN
-F 3 "~" H 8550 1550 50  0001 C CNN
-	1    8550 1550
-	1    0    0    1
-$EndComp
-Wire Wire Line
-	8550 2050 8550 2200
-Connection ~ 9750 2500
-Wire Wire Line
-	8550 1750 8550 1700
-Wire Wire Line
-	9750 1050 9750 2500
-Connection ~ 8550 2500
+P 9750 1550
+F 0 "R_LOWG1" H 9820 1595 50  0000 L CNN
+F 1 "120R" V 9750 1450 50  0000 L CNN
+F 2 "Resistor_SMD:R_0805_2012Metric_Pad1.15x1.40mm_HandSolder" V 9680 1550 50  0001 C CNN
+F 3 "~" H 9750 1550 50  0001 C CNN
+	1    9750 1550
+	-1   0    0    1
+$EndComp
+Wire Wire Line
+	9750 2050 9750 2200
+Wire Wire Line
+	9750 1750 9750 1700
+Wire Wire Line
+	8550 1050 8550 2500
 $Comp
 L Device:R_POT_TRIM RV_TOPG1
@@
 	8550 2500 9200 2500
 Wire Wire Line
-	8550 2200 9100 2200
-Wire Wire Line
-	9100 2200 9100 1900
-Wire Wire Line
-	8700 1900 9100 1900
-Connection ~ 8550 2200
-Wire Wire Line
-	8550 2200 8550 2500
+	9750 2200 9200 2200
+Wire Wire Line
+	9200 2200 9200 1900
+Wire Wire Line
+	9600 1900 9200 1900
+Connection ~ 9750 2200
+Wire Wire Line
+	9750 2200 9750 2500
 $Comp
 L Device:R_POT_Dual_Separate RV_AMP1
@@
 L Device:R_POT_Dual_Separate RV_AMP1
 U 2 1 5BBE484F
-P 8950 1050
-F 0 "RV_AMP1" V 8836 1050 50  0000 C CNN
-F 1 "B10K" V 8747 1050 50  0000 C CNN
-F 2 "PTH901:PTH901" H 8950 1050 50  0001 C CNN
-F 3 "~" H 8950 1050 50  0001 C CNN
-F 4 "652-PTH901-030S-103B" H -550 -2900 50  0001 C CNN "MouserPartNo"
-	2    8950 1050
-	0    -1   1    0
-$EndComp
-Wire Wire Line
-	9750 1050 9300 1050
-Wire Wire Line
-	8550 1050 8800 1050
-Wire Wire Line
-	8550 1400 8550 1050
+P 9350 1050
+F 0 "RV_AMP1" V 9236 1050 50  0000 C CNN
+F 1 "B10K" V 9147 1050 50  0000 C CNN
+F 2 "PTH901:PTH901" H 9350 1050 50  0001 C CNN
+F 3 "~" H 9350 1050 50  0001 C CNN
+F 4 "652-PTH901-030S-103B" H -150 -2900 50  0001 C CNN "MouserPartNo"
+	2    9350 1050
+	0    1    1    0
+$EndComp
+Wire Wire Line
+	8550 1050 9000 1050
+Wire Wire Line
+	9750 1050 9500 1050
+Wire Wire Line
+	9750 1400 9750 1050
 Text HLabel 1150 1600 0    50   Input ~ 0
 SIGIN
-Text HLabel 2950 3350 1    50   Input ~ 0
+Text HLabel 2950 3150 1    50   Input ~ 0
 +12V
-Text HLabel 1350 3350 1    50   Input ~ 0
+Text HLabel 1350 3150 1    50   Input ~ 0
 -12V
-Wire Wire Line
-	2950 3350 2950 3700
-Wire Wire Line
-	1350 3350 1350 3700
 Text HLabel 4150 3600 3    50   Input ~ 0
-GND
+AGND
 Wire Wire Line
 	4150 3600 4150 3400
@@
 	2150 3550 2150 2700
 Wire Wire Line
-	8950 1200 8950 1350
-Wire Wire Line
-	8950 1350 9300 1350
-Wire Wire Line
-	9300 1350 9300 1050
-Connection ~ 9300 1050
-Wire Wire Line
-	9300 1050 9100 1050
+	9350 1200 9350 1350
+Wire Wire Line
+	9350 1350 9000 1350
+Wire Wire Line
+	9000 1350 9000 1050
+Connection ~ 9000 1050
+Wire Wire Line
+	9000 1050 9200 1050
 Wire Wire Line
 	2100 5000 1900 5000
@@
 $EndComp
 Text HLabel 7650 3600 3    50   Input ~ 0
-GND
+AGND
 Wire Wire Line
 	7650 3600 7650 3400
@@
 	9750 3000 9900 3000
 Text HLabel 8550 3600 3    50   Input ~ 0
-GND
+AGND
 Wire Wire Line
 	8550 3600 8550 3100
@@
 Connection ~ 5850 2900
 Text HLabel 4700 3600 3    50   Input ~ 0
-GND
+AGND
 Wire Wire Line
 	4700 3600 4700 3000
@@
 Connection ~ 1900 5000
 Text HLabel 2900 5900 3    50   Input ~ 0
-GND
+AGND
 Wire Wire Line
 	2900 5900 2900 5700
 Text HLabel 6500 5900 3    50   Input ~ 0
-GND
+AGND
 Wire Wire Line
 	6500 5900 6500 5700
 Text HLabel 10500 5900 3    50   Input ~ 0
-GND
+AGND
 Wire Wire Line
 	10500 5900 10500 5700
@@
 F 0 "TP_OFF1" H 2207 2669 50  0000 L CNN
 F 1 "TestPoint" H 2207 2580 50  0000 L CNN
-F 2 "" H 2350 2550 50  0001 C CNN
+F 2 "TestPoint:TestPoint_Pad_D2.0mm" H 2350 2550 50  0001 C CNN
 F 3 "~" H 2350 2550 50  0001 C CNN
 	1    2150 2550
@@
 	2150 2550 2150 2700
 Connection ~ 2150 2700
+$Comp
+L Device:R R_LOFF1
+U 1 1 5BBDB6A3
+P 1350 3450
+F 0 "R_LOFF1" H 950 3500 50  0000 L CNN
+F 1 "220R" H 950 3400 50  0000 L CNN
+F 2 "Resistor_SMD:R_0805_2012Metric_Pad1.15x1.40mm_HandSolder" V 1280 3450 50  0001 C CNN
+F 3 "~" H 1350 3450 50  0001 C CNN
+	1    1350 3450
+	1    0    0    -1
+$EndComp
+$Comp
+L Device:R R_HIOFF1
+U 1 1 5BBDB715
+P 2950 3450
+F 0 "R_HIOFF1" H 3020 3495 50  0000 L CNN
+F 1 "220R" H 3020 3406 50  0000 L CNN
+F 2 "Resistor_SMD:R_0805_2012Metric_Pad1.15x1.40mm_HandSolder" V 2880 3450 50  0001 C CNN
+F 3 "~" H 2950 3450 50  0001 C CNN
+	1    2950 3450
+	1    0    0    -1
+$EndComp
+Wire Wire Line
+	1350 3150 1350 3300
+Wire Wire Line
+	1350 3600 1350 3700
+Wire Wire Line
+	2950 3300 2950 3150
+Wire Wire Line
+	2950 3600 2950 3700
+Connection ~ 8550 2500
+Connection ~ 9750 2500
 $EndSCHEMATC

Commit message: updated HW (output section)
- Switched VFA LM7171 for CFA LT1227 (improved frequency response)
- Removed TL071 from output section
Parts:
- removed C_GAINF1, C_MIXF1, C_MIXIN1: ?, Capacitor_SMD:C_0805_2012Metric_Pad1.15x1.40mm_HandSolder, symbol Device:C
- removed C_MIXBP1: 2.2uF TANT., Capacitor_SMD:C_0805_2012Metric_Pad1.15x1.40mm_HandSolder, symbol Device:CP
- removed C_MIXBP2, C_MIXBP3: 10nF, Capacitor_SMD:C_0805_2012Metric_Pad1.15x1.40mm_HandSolder, symbol Device:C
- removed C_MIXBP4: 2.2pF TANT., Capacitor_SMD:C_0805_2012Metric_Pad1.15x1.40mm_HandSolder, symbol Device:CP
- removed RV_LOWG1: 100R, Potentiometer_THT:Potentiometer_Bourns_3296Y_Vertical, symbol Device:R_POT_TRIM
- removed RV_TOPG1: 10K, Potentiometer_THT:Potentiometer_Bourns_3296Y_Vertical, symbol Device:R_POT_TRIM
- removed R_LOWG1: 120R, Resistor_SMD:R_0805_2012Metric_Pad1.15x1.40mm_HandSolder, symbol Device:R
- removed R_MIXF1: 10K, Resistor_SMD:R_0805_2012Metric_Pad1.15x1.40mm_HandSolder, symbol Device:R
- removed R_TOPG1: 330R, Resistor_SMD:R_0805_2012Metric_Pad1.15x1.40mm_HandSolder, symbol Device:R
- removed U_MIX1: LM7171, Package_SO:SOIC-8_3.9x4.9mm_P1.27mm, symbol Amplifier_Custom:LM7171
- added RF1, RG1: 1k, Resistor_SMD:R_0805_2012Metric_Pad1.15x1.40mm_HandSolder, symbol Device:R
- added RF2: 18K, Resistor_SMD:R_0805_2012Metric_Pad1.15x1.40mm_HandSolder, symbol Device:R
- R_MIX1, R_MIX2: value 10K -> 1K
Connections:
- wire segments 127 -> 78

Commit message: updates
Parts:
- removed C_BUFBP1, C_BUFBP2: 100nF, Capacitor_SMD:C_0805_2012Metric_Pad1.15x1.40mm_HandSolder, symbol Device:C
- removed C_GAINBP1, C_GAINBP4: 2.2uF TANT., Capacitor_SMD:C_0805_2012Metric_Pad1.15x1.40mm_HandSolder, symbol Device:CP
- removed U_BUF1: TL071, Package_SO:SOIC-8_3.9x4.9mm_P1.27mm, symbol Amplifier_Custom:TL071
- removed U_GAIN1: LM7171, Package_SO:SOIC-8_3.9x4.9mm_P1.27mm, symbol Amplifier_Custom:LM7171
- added C_BUFFBP1, C_BUFFBP2: 10nF, Capacitor_SMD:C_0805_2012Metric_Pad1.15x1.40mm_HandSolder, symbol Device:C
- added R_MIX3: 1K, symbol Device:R
- added UBUFF1, UMIX1: LT1227, symbol Amplifier_Custom:LT1227
- renumbered C_GAINBP2 to C_MIXBP1, C_GAINBP3 to C_MIXBP2
Connections:
- net labels added: OFFSETADJUST
- wire segments 78 -> 72

Commit message: update
Parts:
- RF2: value 18K -> 8K2
Changed lines of the file:
@@
 P 8150 2000
 F 0 "RF2" V 7946 2000 50  0000 C CNN
-F 1 "18K" V 8035 2000 50  0000 C CNN
+F 1 "8K2" V 8035 2000 50  0000 C CNN
 F 2 "Resistor_SMD:R_0805_2012Metric_Pad1.15x1.40mm_HandSolder" V 8080 2000 50  0001 C CNN
 F 3 "~" H 8150 2000 50  0001 C CNN
