File: Hardware/OutputSection.sch (KiCad schematic (older format))
At the start: 20 parts

Commit message: board rev b
Parts:
- C_BUFFBP1, C_BUFFBP2, C_MIXBP1, C_MIXBP2: value 10nF -> 100nF
- R_HIOFF1, R_LOFF1: value 220R -> 1K
- R_MIX3: footprint (none) -> Resistor_SMD:R_0805_2012Metric_Pad1.15x1.40mm_HandSolder
- UBUFF1, UMIX1: footprint (none) -> Package_SO:SOIC-8_3.9x4.9mm_P1.27mm
Other:
- note added: "MCU Offset\n"
- note added: "User Gain"
- note added: "User Offset\n"
Changed lines of the file:
@@
 AR Path="/5BBD761F/5BC85CD1" Ref="C_MIXBP1"  Part="1"
 F 0 "C_MIXBP1" H 4350 6750 50  0000 C CNN
-F 1 "10nF" H 4350 6600 50  0000 C CNN
+F 1 "100nF" H 4350 6600 50  0000 C CNN
 F 2 "Capacitor_SMD:C_0805_2012Metric_Pad1.15x1.40mm_HandSolder" H 4638 6500 50  0001 C CNN
 F 3 "~" H 4600 6650 50  0001 C CNN
@@
 AR Path="/5BBD761F/5BC85CDF" Ref="C_MIXBP2"  Part="1"
 F 0 "C_MIXBP2" H 5300 6750 50  0000 C CNN
-F 1 "10nF" H 5350 6600 50  0000 C CNN
+F 1 "100nF" H 5350 6600 50  0000 C CNN
 F 2 "Capacitor_SMD:C_0805_2012Metric_Pad1.15x1.40mm_HandSolder" H 5638 6500 50  0001 C CNN
 F 3 "~" H 5600 6650 50  0001 C CNN
@@
 P 3500 4750
 F 0 "R_LOFF1" H 3100 4800 50  0000 L CNN
-F 1 "220R" H 3100 4700 50  0000 L CNN
+F 1 "1K" H 3100 4700 50  0000 L CNN
 F 2 "Resistor_SMD:R_0805_2012Metric_Pad1.15x1.40mm_HandSolder" V 3430 4750 50  0001 C CNN
 F 3 "~" H 3500 4750 50  0001 C CNN
@@
 P 5100 4750
 F 0 "R_HIOFF1" H 5170 4795 50  0000 L CNN
-F 1 "220R" H 5170 4706 50  0000 L CNN
+F 1 "1K" H 5170 4706 50  0000 L CNN
 F 2 "Resistor_SMD:R_0805_2012Metric_Pad1.15x1.40mm_HandSolder" V 5030 4750 50  0001 C CNN
 F 3 "~" H 5100 4750 50  0001 C CNN
@@
 F 0 "UMIX1" H 8400 3264 50  0000 C CNN
 F 1 "LT1227" H 8400 3175 50  0000 C CNN
-F 2 "" H 8400 2900 50  0001 C CNN
+F 2 "Package_SO:SOIC-8_3.9x4.9mm_P1.27mm" H 8400 2900 50  0001 C CNN
 F 3 "" H 8400 2900 50  0001 C CNN
 	1    8400 2900
@@
 F 0 "UBUFF1" H 2350 3164 50  0000 C CNN
 F 1 "LT1227" H 2350 3075 50  0000 C CNN
-F 2 "" H 2350 2800 50  0001 C CNN
+F 2 "Package_SO:SOIC-8_3.9x4.9mm_P1.27mm" H 2350 2800 50  0001 C CNN
 F 3 "" H 2350 2800 50  0001 C CNN
 	1    2350 2800
@@
 F 0 "UMIX1" V 5191 6200 50  0000 C CNN
 F 1 "LT1227" V 5102 6200 50  0000 C CNN
-F 2 "" H 5100 6200 50  0001 C CNN
+F 2 "Package_SO:SOIC-8_3.9x4.9mm_P1.27mm" H 5100 6200 50  0001 C CNN
 F 3 "" H 5100 6200 50  0001 C CNN
 	2    5100 6200
@@
 AR Path="/5BBD761F/5BC244CA" Ref="C_BUFFBP1"  Part="1"
 F 0 "C_BUFFBP1" H 1350 6750 50  0000 C CNN
-F 1 "10nF" H 1350 6600 50  0000 C CNN
+F 1 "100nF" H 1350 6600 50  0000 C CNN
 F 2 "Capacitor_SMD:C_0805_2012Metric_Pad1.15x1.40mm_HandSolder" H 1638 6500 50  0001 C CNN
 F 3 "~" H 1600 6650 50  0001 C CNN
@@
 AR Path="/5BBD761F/5BC244D0" Ref="C_BUFFBP2"  Part="1"
 F 0 "C_BUFFBP2" H 2300 6750 50  0000 C CNN
-F 1 "10nF" H 2350 6600 50  0000 C CNN
+F 1 "100nF" H 2350 6600 50  0000 C CNN
 F 2 "Capacitor_SMD:C_0805_2012Metric_Pad1.15x1.40mm_HandSolder" H 2638 6500 50  0001 C CNN
 F 3 "~" H 2600 6650 50  0001 C CNN
@@
 F 0 "UBUFF1" V 2191 6200 50  0000 C CNN
 F 1 "LT1227" V 2102 6200 50  0000 C CNN
-F 2 "" H 2100 6200 50  0001 C CNN
+F 2 "Package_SO:SOIC-8_3.9x4.9mm_P1.27mm" H 2100 6200 50  0001 C CNN
 F 3 "" H 2100 6200 50  0001 C CNN
 	2    2100 6200
@@
 F 0 "R_MIX3" H 4370 2495 50  0000 L CNN
 F 1 "1K" H 4370 2406 50  0000 L CNN
-F 2 "" V 4230 2450 50  0001 C CNN
+F 2 "Resistor_SMD:R_0805_2012Metric_Pad1.15x1.40mm_HandSolder" V 4230 2450 50  0001 C CNN
 F 3 "~" H 4300 2450 50  0001 C CNN
 	1    4300 2450
@@
 Wire Wire Line
 	4300 2600 4300 2800
+Text Notes 4425 4575 0    50   ~ 0
+User Offset\n
+Text Notes 1750 1800 0    50   ~ 0
+MCU Offset\n
+Text Notes 5625 2425 0    50   ~ 0
+User Gain
 $EndSCHEMATC

Commit message: updated board layout
Parts:
- removed UBUFF1, UMIX1: LT1227, Package_SO:SOIC-8_3.9x4.9mm_P1.27mm, symbol Amplifier_Custom:LT1227
- added CF2: 2pF, Capacitor_SMD:C_0805_2012Metric_Pad1.15x1.40mm_HandSolder, symbol Device:C
- added C_BUFFBP3: 100nF, Capacitor_SMD:C_0805_2012Metric_Pad1.15x1.40mm_HandSolder, symbol Device:C
- added C_BUFFBP4, C_MIXBP1, C_MIXBP4: 2.2uF, Capacitor_SMD:C_0805_2012Metric_Pad1.15x1.40mm_HandSolder, symbol Device:C
- added U_BUFF1, U_MIX1: LM7171, Package_SO:SOIC-8_3.9x4.9mm_P1.27mm, symbol Amplifier_Custom:LM7171
- C_BUFFBP1: value 100nF -> 2.2uF
- RV_LOWOFF1, RV_UPOFF1: footprint Potentiometer_THT:Potentiometer_Bourns_3296Y_Vertical -> Potentiometer_THT:Potentiometer_Piher_PT-6-V_Vertical
- renumbered C_MIXBP1 to C_MIXBP2, C_MIXBP2 to C_MIXBP3
Connections:
- wire segments 72 -> 92

Commit message: Updated footprints
Parts:
- RV_LOWOFF1, RV_UPOFF1: footprint Potentiometer_THT:Potentiometer_Piher_PT-6-V_Vertical -> Potentiometer_THT:Potentiometer_Piher_PT-6-H_Horizontal
Changed lines of the file:
@@
 F 0 "RV_UPOFF1" V 4650 5000 50  0000 C CNN
 F 1 "100K" V 4550 5000 50  0000 C CNN
-F 2 "Potentiometer_THT:Potentiometer_Piher_PT-6-V_Vertical" H 4800 5000 50  0001 C CNN
+F 2 "Potentiometer_THT:Potentiometer_Piher_PT-6-H_Horizontal" H 4800 5000 50  0001 C CNN
 F 3 "~" H 4800 5000 50  0001 C CNN
 F 4 "652-3296Y-1-104LF" H -650 3650 50  0001 C CNN "MouserPartNo"
@@
 F 0 "RV_LOWOFF1" V 3650 5000 50  0000 C CNN
 F 1 "100K" V 3550 5000 50  0000 C CNN
-F 2 "Potentiometer_THT:Potentiometer_Piher_PT-6-V_Vertical" H 3800 5000 50  0001 C CNN
+F 2 "Potentiometer_THT:Potentiometer_Piher_PT-6-H_Horizontal" H 3800 5000 50  0001 C CNN
 F 3 "~" H 3800 5000 50  0001 C CNN
 F 4 "652-3296Y-1-104LF" H -1650 2950 50  0001 C CNN "MouserPartNo"

Commit message: increased size of board layout to accomodate pot clearance.
Connections:
- net labels added: GND
- net labels removed: AGND
Changed lines of the file:
@@
 $EndComp
 Text HLabel 6850 3500 3    50   Input ~ 0
-AGND
+GND
 Wire Wire Line
 	6850 3500 6850 3300
@@
 	7750 2800 8100 2800
 Text HLabel 7750 3500 3    50   Input ~ 0
-AGND
+GND
 Wire Wire Line
 	7750 3500 7750 3000
@@
 Connection ~ 9250 5000
 Text HLabel 9250 5900 3    50   Input ~ 0
-AGND
+GND
 Wire Wire Line
 	9250 5900 9250 5700
@@
 	4300 3950 4300 4850
 Text HLabel 1800 3700 3    50   Input ~ 0
-AGND
+GND
 Wire Wire Line
 	9050 5000 9250 5000
@@
 Connection ~ 3350 6350
 Text HLabel 3350 7250 3    50   Input ~ 0
-AGND
+GND
 Wire Wire Line
 	3350 7250 3350 7050

Commit message: Reduced size of board width to 90mm
Parts:
- RV_LOWOFF1, RV_UPOFF1: footprint Potentiometer_THT:Potentiometer_Piher_PT-6-H_Horizontal -> Potentiometer_THT:Potentiometer_Piher_PT-6-V_Vertical
Changed lines of the file:
@@
 F 0 "RV_UPOFF1" V 4650 5000 50  0000 C CNN
 F 1 "100K" V 4550 5000 50  0000 C CNN
-F 2 "Potentiometer_THT:Potentiometer_Piher_PT-6-H_Horizontal" H 4800 5000 50  0001 C CNN
+F 2 "Potentiometer_THT:Potentiometer_Piher_PT-6-V_Vertical" H 4800 5000 50  0001 C CNN
 F 3 "~" H 4800 5000 50  0001 C CNN
 F 4 "652-3296Y-1-104LF" H -650 3650 50  0001 C CNN "MouserPartNo"
@@
 F 0 "RV_LOWOFF1" V 3650 5000 50  0000 C CNN
 F 1 "100K" V 3550 5000 50  0000 C CNN
-F 2 "Potentiometer_THT:Potentiometer_Piher_PT-6-H_Horizontal" H 3800 5000 50  0001 C CNN
+F 2 "Potentiometer_THT:Potentiometer_Piher_PT-6-V_Vertical" H 3800 5000 50  0001 C CNN
 F 3 "~" H 3800 5000 50  0001 C CNN
 F 4 "652-3296Y-1-104LF" H -1650 2950 50  0001 C CNN "MouserPartNo"

Commit message: Draft RevA Board
Parts:
- added CF1: 2pF, Capacitor_SMD:C_0805_2012Metric_Pad1.15x1.40mm_HandSolder, symbol Device:C
Connections:
- wire segments 92 -> 96
Changed lines of the file:
@@
 L Device:R RG1
 U 1 1 5BC2C675
-P 1800 3550
-F 0 "RG1" H 1730 3505 50  0000 R CNN
-F 1 "1k" H 1730 3594 50  0000 R CNN
-F 2 "Resistor_SMD:R_0805_2012Metric_Pad1.15x1.40mm_HandSolder" V 1730 3550 50  0001 C CNN
-F 3 "~" H 1800 3550 50  0001 C CNN
-	1    1800 3550
+P 1800 4050
+F 0 "RG1" H 1730 4005 50  0000 R CNN
+F 1 "1k" H 1730 4094 50  0000 R CNN
+F 2 "Resistor_SMD:R_0805_2012Metric_Pad1.15x1.40mm_HandSolder" V 1730 4050 50  0001 C CNN
+F 3 "~" H 1800 4050 50  0001 C CNN
+	1    1800 4050
 	1    0    0    1
 $EndComp
 Wire Wire Line
-	1800 3400 1800 3300
+	1800 3900 1800 3800
 Connection ~ 1800 3300
 Wire Wire Line
@@
 Wire Wire Line
 	4300 3950 4300 4850
-Text HLabel 1800 3700 3    50   Input ~ 0
+Text HLabel 1800 4200 3    50   Input ~ 0
 GND
 Wire Wire Line
@@
 	8800 1350 8800 2000
 Connection ~ 8800 2000
+$Comp
+L Device:C CF1
+U 1 1 5BCAE7B9
+P 2350 3800
+F 0 "CF1" V 2650 3800 50  0000 C CNN
+F 1 "2pF" V 2550 3800 50  0000 C CNN
+F 2 "Capacitor_SMD:C_0805_2012Metric_Pad1.15x1.40mm_HandSolder" H 2388 3650 50  0001 C CNN
+F 3 "~" H 2350 3800 50  0001 C CNN
+	1    2350 3800
+	0    1    1    0
+$EndComp
+Wire Wire Line
+	2200 3800 1800 3800
+Connection ~ 1800 3800
+Wire Wire Line
+	1800 3800 1800 3300
+Wire Wire Line
+	2500 3800 2850 3800
+Wire Wire Line
+	2850 3800 2850 3300
+Connection ~ 2850 3300
 $EndSCHEMATC
